Commit message: Updated paths to stl objects

File: leg_left.urdf (robot description, URDF)
Before this commit: robot leg_left, 7 links, 6 joints
Links:
- link MG996f: geometry collision mesh filename=CAD/MG996.stl scale=0.001 0.001 0.001; visual mesh filename=CAD/MG996.stl scale=0.001 0.001 0.001
- link MG996t: geometry collision mesh filename=CAD/MG996.stl scale=0.001 0.001 0.001; visual mesh filename=CAD/MG996.stl scale=0.001 0.001 0.001
- link base_link: geometry collision mesh filename=CAD/MG996.stl scale=0.001 0.001 0.001; visual mesh filename=CAD/MG996.stl scale=0.001 0.001 0.001
- link coxa: geometry collision mesh filename=CAD/coxa_left.stl scale=0.001 0.001 0.001; visual mesh filename=CAD/coxa_left.stl scale=0.001 0.001 0.001
- link femur: geometry collision mesh filename=CAD/femur_left.stl scale=0.001 0.001 0.001; visual mesh filename=CAD/femur_left.stl scale=0.001 0.001 0.001
- link shield: geometry collision mesh filename=CAD/shield.stl scale=0.001 0.001 0.001; visual mesh filename=CAD/shield.stl scale=0.001 0.001 0.001
- link tibia: geometry collision mesh filename=CAD/tibia_left.stl scale=0.001 0.001 0.001; visual mesh filename=CAD/tibia_left.stl scale=0.001 0.001 0.001

File: leg_right.urdf (robot description, URDF)
Before this commit: robot leg_right, 7 links, 6 joints
Links:
- link MG996f: geometry collision mesh filename=CAD/MG996.stl scale=0.001 0.001 0.001; visual mesh filename=CAD/MG996.stl scale=0.001 0.001 0.001
- link MG996t: geometry collision mesh filename=CAD/MG996.stl scale=0.001 0.001 0.001; visual mesh filename=CAD/MG996.stl scale=0.001 0.001 0.001
- link base_link: geometry collision mesh filename=CAD/MG996.stl scale=0.001 0.001 0.001; visual mesh filename=CAD/MG996.stl scale=0.001 0.001 0.001
- link coxa: geometry collision mesh filename=CAD/coxa_right.stl scale=0.001 0.001 0.001; visual mesh filename=CAD/coxa_right.stl scale=0.001 0.001 0.001
- link femur: geometry collision mesh filename=CAD/femur_right.stl scale=0.001 0.001 0.001; visual mesh filename=CAD/femur_right.stl scale=0.001 0.001 0.001
- link shield: geometry collision mesh filename=CAD/shield.stl scale=0.001 0.001 0.001; visual mesh filename=CAD/shield.stl scale=0.001 0.001 0.001
- link tibia: geometry collision mesh filename=CAD/tibia_right.stl scale=0.001 0.001 0.001; visual mesh filename=CAD/tibia_right.stl scale=0.001 0.001 0.001
