Commit message: Now we have two URDF: one with all the details and the other one with only the bare minimum

File: hexapod_bare_minimum.urdf (robot description, URDF)
Before this commit: robot hexapod, 50 links, 49 joints
Links:
- removed link bottom_plate
- removed link electronics_layer_1
- removed link electronics_layer_2
- removed link leg1_shield
- removed link leg2_shield
- removed link leg3_shield
- removed link leg4_shield
- removed link leg5_shield
- removed link leg6_shield
- removed link spacer_1
- removed link spacer_2
- removed link spacer_3
- removed link spacer_4
Joints:
- removed joint base_bottom_plate
- removed joint bottom_plate_layer_1
- removed joint layer_1_spacer_1
- removed joint layer_1_spacer_2
- removed joint layer_1_spacer_3
- removed joint layer_1_spacer_4
- removed joint leg1_tibia_shield
- removed joint leg2_tibia_shield
- removed joint leg3_tibia_shield
- removed joint leg4_tibia_shield
- removed joint leg5_tibia_shield
- removed joint leg6_tibia_shield
- removed joint spacer_1_layer_2
