Commit message: Hardware update

File: hexapod_bare_metal.urdf (robot description, URDF)
Before this commit: robot hexapod, 62 links, 61 joints
Links:
- removed link bottom_plate
- removed link electronics_layer_1
- removed link electronics_layer_2
- removed link spacer_1
- removed link spacer_2
- removed link spacer_3
- removed link spacer_4
Joints:
- removed joint base_bottom_plate
- removed joint bottom_plate_electronics_layer_1
- removed joint electronics_layer_1_spacer_1
- removed joint electronics_layer_1_spacer_2
- removed joint electronics_layer_1_spacer_3
- removed joint electronics_layer_1_spacer_4
- removed joint spacer_2_electronics_layer_2

File: leg_left.urdf (robot description, URDF)
Before this commit: robot leg_left, 7 links, 6 joints
Links:
- removed link MG996f
- removed link MG996t
- removed link coxa
- removed link femur
- removed link shield
- removed link tibia
- added link leg_6_MG996R_f, mass 0.207953278714177; collision mesh filename=CAD/MG996R.stl scale=0.001 0.001 0.001; visual mesh filename=CAD/MG996R.stl scale=0.001 0.001 0.001
- added link leg_6_MG996R_t, mass 0.207953278714177; collision mesh filename=CAD/MG996R.stl scale=0.001 0.001 0.001; visual mesh filename=CAD/MG996R.stl scale=0.001 0.001 0.001
- added link leg_6_coxa_a, mass 0.03329037594662584; collision mesh filename=CAD/coxa_a_left.stl scale=0.001 0.001 0.001; visual mesh filename=CAD/coxa_a_left.stl scale=0.001 0.001 0.001
- added link leg_6_coxa_b, mass 0.044908366157452306; collision mesh filename=CAD/coxa_b_left.stl scale=0.001 0.001 0.001; visual mesh filename=CAD/coxa_b_left.stl scale=0.001 0.001 0.001
- added link leg_6_femur_a, mass 0.06532641332455366; collision mesh filename=CAD/femur_a_left.stl scale=0.001 0.001 0.001; visual mesh filename=CAD/femur_a_left.stl scale=0.001 0.001 0.001
- added link leg_6_femur_b, mass 0.0800214310563922; collision mesh filename=CAD/femur_b_left.stl scale=0.001 0.001 0.001; visual mesh filename=CAD/femur_b_left.stl scale=0.001 0.001 0.001
- added link leg_6_femur_c, mass 0.04839907214825549; collision mesh filename=CAD/femur_c_left.stl scale=0.001 0.001 0.001; visual mesh filename=CAD/femur_c_left.stl scale=0.001 0.001 0.001
- added link leg_6_tibia, mass 0.10828707727885012; collision mesh filename=CAD/tibia_left.stl scale=0.001 0.001 0.001; visual mesh filename=CAD/tibia_left.stl scale=0.001 0.001 0.001
- link base_link: mass 0.20641808912389753 -> 0.207953278714177; geometry collision mesh filename=CAD/MG996R.stl scale=0.001 0.001 0.001; visual mesh filename=CAD/MG996R.stl scale=0.001 0.001 0.001
Joints:
- removed joint MG996t_tibia_fixed
- removed joint coxa_MG996f_fixed
- removed joint coxa_joint
- removed joint femur_joint
- removed joint tibia_joint
- removed joint tibia_shield_fixed
- added joint leg_6_MG996R_f_coxa_a: type fixed, parent leg_6_MG996R_f, child leg_6_coxa_a, origin xyz=0.0494 -1.7763568394002505e-17 0.0 rpy=-2.4442543409198012e-32 -1.5707963267948966 0
- added joint leg_6_MG996R_t_tibia: type fixed, parent leg_6_MG996R_t, child leg_6_tibia, origin xyz=0.0027462499999999857 -0.04668051 0.005250000000000004 rpy=6.289234938331016e-17 5.592845782213298e-17 5.551115123125774e-17
- added joint leg_6_coxa_b_MG996R_f: type fixed, parent leg_6_coxa_b, child leg_6_MG996R_f, origin xyz=0.02916816000000001 -0.03906765 -0.00535 rpy=3.141592653589793 -1.5707963267948966 0
- added joint leg_6_coxa_joint: type revolute, parent base_link, child leg_6_coxa_b, origin xyz=0.028425689999999997 0.021001069999999997 0.031066209999999997 rpy=-3.141592653589793 -0.0 1.251344390463166e-32, axis 0.0 6.162975822039155e-33 1.0, limit lower=-1.570796 upper=1.570796 effort=1000000 velocity=1000000
- added joint leg_6_femur_a_femur_b: type fixed, parent leg_6_femur_a, child leg_6_femur_b, origin xyz=0.0007071000000000005 0.000707109999999993 0.057705780000000005 rpy=3.141592653589793 -5.59284578221332e-17 -5.551115123125784e-17
- added joint leg_6_femur_b_femur_c: type fixed, parent leg_6_femur_b, child leg_6_femur_c, origin xyz=-0.03075914 0.030759150000000002 0.0 rpy=-3.141592653589793 1.59199441504844e-17 -5.551115123125784e-17
- added joint leg_6_femur_joint: type revolute, parent leg_6_MG996R_f, child leg_6_femur_a, origin xyz=0.03495 -0.025679440000000008 0.01825481999999999 rpy=3.141592653589793 -1.5707963267948966 0, axis -0.707107 -0.707107 1.4803983593078296e-34, limit lower=-2.356194 upper=0.785398 effort=1000000 velocity=1000000
- added joint leg_6_tibia_joint: type revolute, parent leg_6_femur_a, child leg_6_MG996R_t, origin xyz=0.020918530000000005 -0.020918540000000013 0.06344154 rpy=-6.289234938331015e-17 -5.59284578221332e-17 -5.551115123125784e-17, axis -0.7071069999999999 -0.7071069999999999 -2.4934463508646154e-17, limit lower=-1.570796 upper=1.570796 effort=1000000 velocity=1000000

File: leg_right.urdf (robot description, URDF)
Before this commit: robot leg_right, 7 links, 6 joints
Links:
- removed link MG996f
- removed link MG996t
- removed link coxa
- removed link femur
- removed link shield
- removed link tibia
- added link leg_1_MG996R_f, mass 0.207953278714177; collision mesh filename=CAD/MG996R.stl scale=0.001 0.001 0.001; visual mesh filename=CAD/MG996R.stl scale=0.001 0.001 0.001
- added link leg_1_MG996R_t, mass 0.207953278714177; collision mesh filename=CAD/MG996R.stl scale=0.001 0.001 0.001; visual mesh filename=CAD/MG996R.stl scale=0.001 0.001 0.001
- added link leg_1_coxa_a, mass 0.03329037594662584; collision mesh filename=CAD/coxa_a_right.stl scale=0.001 0.001 0.001; visual mesh filename=CAD/coxa_a_right.stl scale=0.001 0.001 0.001
- added link leg_1_coxa_b, mass 0.04490836615745227; collision mesh filename=CAD/leg_1_coxa_b.stl scale=0.001 0.001 0.001; visual mesh filename=CAD/coxa_b_right.stl scale=0.001 0.001 0.001
- added link leg_1_femur_a, mass 0.06532641332455354; collision mesh filename=CAD/femur_a_right.stl scale=0.001 0.001 0.001; visual mesh filename=CAD/femur_a_right.stl scale=0.001 0.001 0.001
- added link leg_1_femur_b, mass 0.0800214310563922; collision mesh filename=CAD/femur_b_right.stl scale=0.001 0.001 0.001; visual mesh filename=CAD/femur_b_right.stl scale=0.001 0.001 0.001
- added link leg_1_femur_c, mass 0.048399072148255506; collision mesh filename=CAD/femur_c_right.stl scale=0.001 0.001 0.001; visual mesh filename=CAD/femur_c_right.stl scale=0.001 0.001 0.001
- added link leg_1_tibia, mass 0.10828707727885009; collision mesh filename=CAD/tibia_right.stl scale=0.001 0.001 0.001; visual mesh filename=CAD/tibia_right.stl scale=0.001 0.001 0.001
- link base_link: mass 0.20641808912389753 -> 0.207953278714177; geometry collision mesh filename=CAD/MG996R.stl scale=0.001 0.001 0.001; visual mesh filename=CAD/MG996R.stl scale=0.001 0.001 0.001
Joints:
- removed joint MG996t_tibia_fixed
- removed joint coxa_MG996f_fixed
- removed joint coxa_joint
- removed joint femur_joint
- removed joint tibia_joint
- removed joint tibia_shield_fixed
- added joint leg_1_MG996R_f_coxa_a: type fixed, parent leg_1_MG996R_f, child leg_1_coxa_a, origin xyz=0.0494 0.0 0.0 rpy=6.704561300464011e-33 1.5707963267948966 0
- added joint leg_1_MG996R_t_tibia: type fixed, parent leg_1_MG996R_t, child leg_1_tibia, origin xyz=0.033881879999999996 -0.013446489999999986 -0.005250000000000004 rpy=3.141592653589793 -1.6337250741359945e-17 5.551115123125788e-17
- added joint leg_1_coxa_b_MG996R_f: type fixed, parent leg_1_coxa_b, child leg_1_MG996R_f, origin xyz=-0.02916816000000001 -0.03906765 -0.00535 rpy=6.626416783217546e-33 -1.5707963267948966 0
- added joint leg_1_coxa_joint: type revolute, parent base_link, child leg_1_coxa_b, origin xyz=-0.028425689999999997 0.021001069999999997 0.031066209999999997 rpy=3.141592653589793 -0.0 3.0033433937731107e-33, axis 0.0 0.0 1.0, limit lower=-1.570796 upper=1.570796 effort=1000000 velocity=1000000
- added joint leg_1_femur_a_femur_b: type fixed, parent leg_1_femur_a, child leg_1_femur_b, origin xyz=-0.0007071000000000005 0.000707109999999993 0.04770578 rpy=-3.141592653589793 1.6337250741359954e-17 -5.551115123125783e-17
- added joint leg_1_femur_b_femur_c: type fixed, parent leg_1_femur_b, child leg_1_femur_c, origin xyz=0.03075914000000001 0.030759150000000002 0.0 rpy=3.141592653589793 -0.0 -7.002961686799377e-34
- added joint leg_1_femur_joint: type revolute, parent leg_1_MG996R_f, child leg_1_femur_a, origin xyz=0.03495 0.025679440000000008 0.01825481999999999 rpy=6.704561300464011e-33 1.5707963267948966 0, axis 0.707107 -0.707107 1.999343393356845e-32, limit lower=-0.785398 upper=2.356194 effort=1000000 velocity=1000000
- added joint leg_1_tibia_joint: type revolute, parent leg_1_femur_a, child leg_1_MG996R_t, origin xyz=-0.020918530000000005 -0.020918540000000013 0.06344154 rpy=4.0156312877350055e-17 1.6337250741359954e-17 -5.551115123125783e-17, axis -0.707107 0.707107 -1.8398022027031245e-17, limit lower=-1.570796 upper=1.570796 effort=1000000 velocity=1000000
