Commit message: Fixed typo

File: hexapod.urdf (robot description, URDF)
Before this commit: robot hexapod, 62 links, 61 joints
Links:
- link leg_1_coxa_b: geometry collision mesh filename=CAD/coxa_b_right.stl scale=0.001 0.001 0.001; visual mesh filename=CAD/coxa_b_right.stl scale=0.001 0.001 0.001

File: hexapod_bare_metal.urdf (robot description, URDF)
Before this commit: robot hexapod, 55 links, 54 joints
Links:
- link leg_1_coxa_b: geometry collision mesh filename=CAD/coxa_b_right.stl scale=0.001 0.001 0.001; visual mesh filename=CAD/coxa_b_right.stl scale=0.001 0.001 0.001

File: leg_right.urdf (robot description, URDF)
Before this commit: robot hexapod, 9 links, 8 joints
Links:
- link leg_1_coxa_b: geometry collision mesh filename=CAD/coxa_b_right.stl scale=0.001 0.001 0.001; visual mesh filename=CAD/coxa_b_right.stl scale=0.001 0.001 0.001

Commit message: New hexapod version

File: hexapod.urdf (robot description, URDF)
Before this commit: robot hexapod, 62 links, 61 joints
Links:
- removed link bottom_plate
- removed link electronics_layer_1
- removed link electronics_layer_2
- removed link leg_1_MG996R_c
- removed link leg_1_MG996R_f
- removed link leg_1_MG996R_t
- removed link leg_1_coxa_a
- removed link leg_1_coxa_b
- removed link leg_1_femur_a
- removed link leg_1_femur_b
- removed link leg_1_femur_c
- removed link leg_2_MG996R_c
- removed link leg_2_MG996R_f
- removed link leg_2_MG996R_t
- removed link leg_2_coxa_a
- removed link leg_2_coxa_b
- removed link leg_2_femur_a
- removed link leg_2_femur_b
- removed link leg_2_femur_c
- removed link leg_3_MG996R_c
- removed link leg_3_MG996R_f
- removed link leg_3_MG996R_t
- removed link leg_3_coxa_a
- removed link leg_3_coxa_b
- removed link leg_3_femur_a
- removed link leg_3_femur_b
- removed link leg_3_femur_c
- removed link leg_4_MG996R_c
- removed link leg_4_MG996R_f
- removed link leg_4_MG996R_t
- removed link leg_4_coxa_a
- removed link leg_4_coxa_b
- removed link leg_4_femur_a
- removed link leg_4_femur_b
- removed link leg_4_femur_c
- removed link leg_5_MG996R_c
- removed link leg_5_MG996R_f
- removed link leg_5_MG996R_t
- removed link leg_5_coxa_a
- removed link leg_5_coxa_b
- removed link leg_5_femur_a
- removed link leg_5_femur_b
- removed link leg_5_femur_c
- removed link leg_6_MG996R_c
- removed link leg_6_MG996R_f
- removed link leg_6_MG996R_t
- removed link leg_6_coxa_a
- removed link leg_6_coxa_b
- removed link leg_6_femur_a
- removed link leg_6_femur_b
- removed link leg_6_femur_c
- removed link spacer_1
- removed link spacer_2
- removed link spacer_3
- removed link spacer_4
- added link leg_1_MG996R_coxa, mass 0.20795327871559424; collision mesh filename=CAD/MG996R.stl scale=0.001 0.001 0.001; visual mesh filename=CAD/MG996R.stl scale=0.001 0.001 0.001
- added link leg_1_MG996R_femur, mass 0.20795327871559424; collision mesh filename=CAD/MG996R.stl scale=0.001 0.001 0.001; visual mesh filename=CAD/MG996R.stl scale=0.001 0.001 0.001
- added link leg_1_MG996R_tibia, mass 0.20795327871559424; collision mesh filename=CAD/MG996R.stl scale=0.001 0.001 0.001; visual mesh filename=CAD/MG996R.stl scale=0.001 0.001 0.001
- added link leg_1_coxa, mass 0.23210805328252043; collision mesh filename=CAD/coxa.stl scale=0.001 0.001 0.001; visual mesh filename=CAD/coxa.stl scale=0.001 0.001 0.001
- added link leg_1_femur, mass 0.1615808293904576; collision mesh filename=CAD/femur.stl scale=0.001 0.001 0.001; visual mesh filename=CAD/femur.stl scale=0.001 0.001 0.001
- added link leg_2_MG996R_coxa, mass 0.20795327871559424; collision mesh filename=CAD/MG996R.stl scale=0.001 0.001 0.001; visual mesh filename=CAD/MG996R.stl scale=0.001 0.001 0.001
- added link leg_2_MG996R_femur, mass 0.20795327871559424; collision mesh filename=CAD/MG996R.stl scale=0.001 0.001 0.001; visual mesh filename=CAD/MG996R.stl scale=0.001 0.001 0.001
- added link leg_2_MG996R_tibia, mass 0.20795327871559424; collision mesh filename=CAD/MG996R.stl scale=0.001 0.001 0.001; visual mesh filename=CAD/MG996R.stl scale=0.001 0.001 0.001
- added link leg_2_coxa, mass 0.23210805328252054; collision mesh filename=CAD/coxa.stl scale=0.001 0.001 0.001; visual mesh filename=CAD/coxa.stl scale=0.001 0.001 0.001
- added link leg_2_femur, mass 0.1615808293904576; collision mesh filename=CAD/femur.stl scale=0.001 0.001 0.001; visual mesh filename=CAD/femur.stl scale=0.001 0.001 0.001
- added link leg_3_MG996R_coxa, mass 0.20795327871559424; collision mesh filename=CAD/MG996R.stl scale=0.001 0.001 0.001; visual mesh filename=CAD/MG996R.stl scale=0.001 0.001 0.001
- added link leg_3_MG996R_femur, mass 0.20795327871559424; collision mesh filename=CAD/MG996R.stl scale=0.001 0.001 0.001; visual mesh filename=CAD/MG996R.stl scale=0.001 0.001 0.001
- added link leg_3_MG996R_tibia, mass 0.20795327871559424; collision mesh filename=CAD/MG996R.stl scale=0.001 0.001 0.001; visual mesh filename=CAD/MG996R.stl scale=0.001 0.001 0.001
- added link leg_3_coxa, mass 0.23210805328252054; collision mesh filename=CAD/coxa.stl scale=0.001 0.001 0.001; visual mesh filename=CAD/coxa.stl scale=0.001 0.001 0.001
- added link leg_3_femur, mass 0.1615808293904576; collision mesh filename=CAD/femur.stl scale=0.001 0.001 0.001; visual mesh filename=CAD/femur.stl scale=0.001 0.001 0.001
- added link leg_4_MG996R_coxa, mass 0.20795327871559424; collision mesh filename=CAD/MG996R.stl scale=0.001 0.001 0.001; visual mesh filename=CAD/MG996R.stl scale=0.001 0.001 0.001
- added link leg_4_MG996R_femur, mass 0.20795327871559424; collision mesh filename=CAD/MG996R.stl scale=0.001 0.001 0.001; visual mesh filename=CAD/MG996R.stl scale=0.001 0.001 0.001
- added link leg_4_MG996R_tibia, mass 0.20795327871559424; collision mesh filename=CAD/MG996R.stl scale=0.001 0.001 0.001; visual mesh filename=CAD/MG996R.stl scale=0.001 0.001 0.001
- added link leg_4_coxa, mass 0.23210805328252054; collision mesh filename=CAD/coxa.stl scale=0.001 0.001 0.001; visual mesh filename=CAD/coxa.stl scale=0.001 0.001 0.001
- added link leg_4_femur, mass 0.1615808293904576; collision mesh filename=CAD/femur.stl scale=0.001 0.001 0.001; visual mesh filename=CAD/femur.stl scale=0.001 0.001 0.001
- added link leg_5_MG996R_coxa, mass 0.20795327871559424; collision mesh filename=CAD/MG996R.stl scale=0.001 0.001 0.001; visual mesh filename=CAD/MG996R.stl scale=0.001 0.001 0.001
- added link leg_5_MG996R_femur, mass 0.20795327871559424; collision mesh filename=CAD/MG996R.stl scale=0.001 0.001 0.001; visual mesh filename=CAD/MG996R.stl scale=0.001 0.001 0.001
- added link leg_5_MG996R_tibia, mass 0.20795327871559424; collision mesh filename=CAD/MG996R.stl scale=0.001 0.001 0.001; visual mesh filename=CAD/MG996R.stl scale=0.001 0.001 0.001
- added link leg_5_coxa, mass 0.23210805328252054; collision mesh filename=CAD/coxa.stl scale=0.001 0.001 0.001; visual mesh filename=CAD/coxa.stl scale=0.001 0.001 0.001
- added link leg_5_femur, mass 0.1615808293904576; collision mesh filename=CAD/femur.stl scale=0.001 0.001 0.001; visual mesh filename=CAD/femur.stl scale=0.001 0.001 0.001
- added link leg_6_MG996R_coxa, mass 0.20795327871559424; collision mesh filename=CAD/MG996R.stl scale=0.001 0.001 0.001; visual mesh filename=CAD/MG996R.stl scale=0.001 0.001 0.001
- added link leg_6_MG996R_femur, mass 0.20795327871559424; collision mesh filename=CAD/MG996R.stl scale=0.001 0.001 0.001; visual mesh filename=CAD/MG996R.stl scale=0.001 0.001 0.001
- added link leg_6_MG996R_tibia, mass 0.20795327871559424; collision mesh filename=CAD/MG996R.stl scale=0.001 0.001 0.001; visual mesh filename=CAD/MG996R.stl scale=0.001 0.001 0.001
- added link leg_6_coxa, mass 0.23210805328252054; collision mesh filename=CAD/coxa.stl scale=0.001 0.001 0.001; visual mesh filename=CAD/coxa.stl scale=0.001 0.001 0.001
- added link leg_6_femur, mass 0.1615808293904576; collision mesh filename=CAD/femur.stl scale=0.001 0.001 0.001; visual mesh filename=CAD/femur.stl scale=0.001 0.001 0.001
- link base: mass 0.6789580603579961 -> 0.5452508805768645
- link leg_1_tibia: mass 0.10828707727885009 -> 0.2763071087572843; geometry collision mesh filename=CAD/tibia.stl scale=0.001 0.001 0.001; visual mesh filename=CAD/tibia.stl scale=0.001 0.001 0.001
- link leg_2_tibia: mass 0.10828707727885009 -> 0.2763071087572843; geometry collision mesh filename=CAD/tibia.stl scale=0.001 0.001 0.001; visual mesh filename=CAD/tibia.stl scale=0.001 0.001 0.001
- link leg_3_tibia: mass 0.10828707727885009 -> 0.2763071087572843; geometry collision mesh filename=CAD/tibia.stl scale=0.001 0.001 0.001; visual mesh filename=CAD/tibia.stl scale=0.001 0.001 0.001
- link leg_4_tibia: mass 0.10828707727885012 -> 0.2763071087572843; geometry collision mesh filename=CAD/tibia.stl scale=0.001 0.001 0.001; visual mesh filename=CAD/tibia.stl scale=0.001 0.001 0.001
- link leg_5_tibia: mass 0.10828707727885012 -> 0.2763071087572843; geometry collision mesh filename=CAD/tibia.stl scale=0.001 0.001 0.001; visual mesh filename=CAD/tibia.stl scale=0.001 0.001 0.001
- link leg_6_tibia: mass 0.10828707727885012 -> 0.2763071087572843; geometry collision mesh filename=CAD/tibia.stl scale=0.001 0.001 0.001; visual mesh filename=CAD/tibia.stl scale=0.001 0.001 0.001
Joints:
- removed joint base_bottom_plate
- removed joint base_leg_1_MG996R_c
- removed joint base_leg_2_MG996R_c
- removed joint base_leg_3_MG996R_c
- removed joint base_leg_4_MG996R_c
- removed joint base_leg_5_MG996R_c
- removed joint base_leg_6_MG996R_c
- removed joint bottom_plate_electronics_layer_1
- removed joint electronics_layer_1_spacer_1
- removed joint electronics_layer_1_spacer_2
- removed joint electronics_layer_1_spacer_3
- removed joint electronics_layer_1_spacer_4
- removed joint leg_1_MG996R_f_coxa_a
- removed joint leg_1_MG996R_t_tibia
- removed joint leg_1_coxa_b_MG996R_f
- removed joint leg_1_coxa_joint
- removed joint leg_1_femur_a_femur_b
- removed joint leg_1_femur_b_femur_c
- removed joint leg_1_femur_joint
- removed joint leg_1_tibia_joint
- removed joint leg_2_MG996R_f_coxa_a
- removed joint leg_2_MG996R_t_tibia
- removed joint leg_2_coxa_b_MG996R_f
- removed joint leg_2_coxa_joint
- removed joint leg_2_femur_a_femur_b
- removed joint leg_2_femur_b_femur_c
- removed joint leg_2_femur_joint
- removed joint leg_2_tibia_joint
- removed joint leg_3_MG996R_f_coxa_a
- removed joint leg_3_MG996R_t_tibia
- removed joint leg_3_coxa_b_MG996R_f
- removed joint leg_3_coxa_joint
- removed joint leg_3_femur_a_femur_b
- removed joint leg_3_femur_b_femur_c
- removed joint leg_3_femur_joint
- removed joint leg_3_tibia_joint
- removed joint leg_4_MG996R_f_coxa_a
- removed joint leg_4_MG996R_t_tibia
- removed joint leg_4_coxa_b_MG996R_f
- removed joint leg_4_coxa_joint
- removed joint leg_4_femur_a_femur_b
- removed joint leg_4_femur_b_femur_c
- removed joint leg_4_femur_joint
- removed joint leg_4_tibia_joint
- removed joint leg_5_MG996R_f_coxa_a
- removed joint leg_5_MG996R_t_tibia
- removed joint leg_5_coxa_b_MG996R_f
- removed joint leg_5_coxa_joint
- removed joint leg_5_femur_a_femur_b
- removed joint leg_5_femur_b_femur_c
- removed joint leg_5_femur_joint
- removed joint leg_5_tibia_joint
- removed joint leg_6_MG996R_f_coxa_a
- removed joint leg_6_MG996R_t_tibia
- removed joint leg_6_coxa_b_MG996R_f
- removed joint leg_6_coxa_joint
- removed joint leg_6_femur_a_femur_b
- removed joint leg_6_femur_b_femur_c
- removed joint leg_6_femur_joint
- removed joint leg_6_tibia_joint
- removed joint spacer_2_electronics_layer_2
- added joint base_leg_1: type fixed, parent base, child leg_1_MG996R_coxa, origin xyz=0.03687244 0.05481281999999997 -3.3306690738754402e-18 rpy=1.5777218104420236e-30 3.155443620884054e-30 3.141592653589793
- added joint base_leg_2: type fixed, parent base, child leg_2_MG996R_coxa, origin xyz=0.03713499999999998 0.005249999999999989 -3.3306690738753613e-18 rpy=1.5777218104420236e-30 3.155443620884054e-30 3.141592653589793
- added joint base_leg_3: type fixed, parent base, child leg_3_MG996R_coxa, origin xyz=0.03687243999999997 -0.054812819999999984 -3.3306690738752677e-18 rpy=1.5777218104420236e-30 3.155443620884054e-30 3.141592653589793
- added joint base_leg_4: type fixed, parent base, child leg_4_MG996R_coxa, origin xyz=-0.02944782 -0.06223743999999996 -3.330669073875465e-18 rpy=1.5777218104420236e-30 3.155443620884054e-30 3.141592653589793
- added joint base_leg_5: type fixed, parent base, child leg_5_MG996R_coxa, origin xyz=-0.03713499999999998 -0.005249999999999989 -3.3306690738755793e-18 rpy=1.5777218104420236e-30 3.155443620884054e-30 3.141592653589793
- added joint base_leg_6: type fixed, parent base, child leg_6_MG996R_coxa, origin xyz=-0.03687243999999997 0.054812819999999984 -3.330669073875673e-18 rpy=1.5777218104420236e-30 3.155443620884054e-30 3.141592653589793
- added joint leg_1_coxa: type continuous, parent leg_1_MG996R_coxa, child leg_1_coxa, origin xyz=-0.02100107 -0.028425689999999993 0.03106621 rpy=9.860761315262648e-32 -0.0 9.80394874699742e-31, axis -0.0 -9.860761315262648e-32 -1.0
- added joint leg_1_femur: type continuous, parent leg_1_coxa, child leg_1_MG996R_femur, origin xyz=-0.057629200000000005 -0.027223610000000013 -0.0215 rpy=-7.942107605087364e-16 0.7853981633974434 3.1415926535897927, axis 0.5000001547244789 -0.7071069999999999 0.5000001547244733
- added joint leg_1_tibia: type continuous, parent leg_1_MG996R_tibia, child leg_1_tibia, origin xyz=-0.011749440000000017 -0.03218482000000002 -0.005250000000000001 rpy=3.141592653589793 -2.455971556515381e-28 1.5777218104420236e-30, axis 0.707107 -0.707107 -2.4656518234403854e-29
- added joint leg_2_coxa: type continuous, parent leg_2_MG996R_coxa, child leg_2_coxa, origin xyz=-0.03495 0.00525 0.03106621 rpy=0.0 1.9721522630525295e-31 5.593936126472314e-33, axis 1.9721522630525295e-31 0.0 -0.9999999999999999
- added joint leg_2_femur: type continuous, parent leg_2_coxa, child leg_2_MG996R_femur, origin xyz=-0.06000000000000001 0.0215 -0.021500000000000005 rpy=-7.422322462533451e-16 0.7853981633974433 3.1415926535897927, axis 3.711161231266726e-16 -1.0 -3.711161231266763e-16
- added joint leg_2_tibia: type continuous, parent leg_2_MG996R_tibia, child leg_2_tibia, origin xyz=0.014450000000000003 -0.03106621 -0.005250000000000001 rpy=-3.141592653589793 -1.977608157853436e-31 -1.5777218104420236e-30, axis 0.0 -0.9999999999999999 -1.5777218104420236e-30
- added joint leg_3_coxa: type continuous, parent leg_3_MG996R_coxa, child leg_3_coxa, origin xyz=-0.02100107 0.028425689999999993 0.03106621 rpy=0.0 -1.9721522630525295e-31 -3.390661277973094e-45, axis -1.9721522630525295e-31 0.0 -0.9999999999999999
- added joint leg_3_femur: type continuous, parent leg_3_coxa, child leg_3_MG996R_femur, origin xyz=-0.027223610000000002 0.05762920000000001 -0.02150000000000001 rpy=-7.080538306756965e-16 0.7853981633974434 3.1415926535897927, axis -0.5000001547244785 -0.707107 -0.5000001547244738
- added joint leg_3_tibia: type continuous, parent leg_3_MG996R_tibia, child leg_3_tibia, origin xyz=0.03218482000000002 -0.01174944 -0.00525 rpy=-3.141592653589793 -3.1507118818835715e-28 -1.577721810442024e-30, axis -0.707107 -0.7071069999999999 3.247757628198293e-29
- added joint leg_4_coxa: type continuous, parent leg_4_MG996R_coxa, child leg_4_coxa, origin xyz=0.028425690000000003 0.021001069999999997 0.03106621 rpy=-1.9721522630525295e-31 -1.9721522630525295e-31 -1.4971863295389187e-31, axis -1.9721522630525295e-31 1.9721522630525295e-31 -1.0
- added joint leg_4_femur: type continuous, parent leg_4_coxa, child leg_4_MG996R_femur, origin xyz=0.057629200000000005 0.027223610000000013 -0.0215 rpy=-6.469461358014946e-16 0.7853981633974433 3.1415926535897927, axis -0.500000154724479 0.707107 -0.5000001547244732
- added joint leg_4_tibia: type continuous, parent leg_4_MG996R_tibia, child leg_4_tibia, origin xyz=0.048377570000000016 -0.001049199999999999 -0.005250000000000001 rpy=3.141592653589793 -3.392272815550781e-28 -4.592132580746781e-86, axis -0.707107 0.707107 4.337944936001927e-29
- added joint leg_5_coxa: type continuous, parent leg_5_MG996R_coxa, child leg_5_coxa, origin xyz=0.03495 -0.00525 0.03106621 rpy=-9.860761315262648e-32 -0.0 1.0138806576528696e-32, axis 0.0 9.860761315262648e-32 -1.0
- added joint leg_5_femur: type continuous, parent leg_5_coxa, child leg_5_MG996R_femur, origin xyz=0.06000000000000001 -0.0215 -0.0215 rpy=-7.422322462533452e-16 0.7853981633974433 3.1415926535897927, axis -3.711161231266728e-16 1.0 3.711161231266763e-16
- added joint leg_5_tibia: type continuous, parent leg_5_MG996R_tibia, child leg_5_tibia, origin xyz=0.03495000000000001 0.03106621 -0.005250000000000001 rpy=-3.141592653589793 9.729700613564994e-32 1.5777218104420236e-30, axis -1.5777218104420236e-30 0.9999999999999999 0.0
- added joint leg_6_coxa: type continuous, parent leg_6_MG996R_coxa, child leg_6_coxa, origin xyz=0.02100107 -0.028425689999999993 0.03106621 rpy=1.97215226305253e-31 -0.0 1.6819919341129893e-45, axis 0.0 -1.9721522630525295e-31 -0.9999999999999999
- added joint leg_6_femur: type continuous, parent leg_6_coxa, child leg_6_MG996R_femur, origin xyz=0.027223610000000002 -0.05762920000000003 -0.021500000000000005 rpy=-6.349165004021658e-16 0.7853981633974433 3.1415926535897927, axis 0.5000001547244782 0.707107 0.5000001547244738
- added joint leg_6_tibia: type continuous, parent leg_6_MG996R_tibia, child leg_6_tibia, origin xyz=0.0027462500000000035 0.04668052000000001 -0.005250000000000001 rpy=-3.141592653589793 -3.640945256296552e-28 -1.577721810442024e-30, axis 0.707107 0.7071069999999999 -4.4724723353636215e-29
- added joint leg_leg_1_MG996R_femur: type fixed, parent leg_1_MG996R_femur, child leg_1_femur, origin xyz=-0.01904579387203917 0.011749440000000017 -0.02647041507449769 rpy=-5.248374545410791e-16 0.7853981633974433 -3.141592653589793
- added joint leg_leg_1_femur_MG996R: type fixed, parent leg_1_femur, child leg_1_MG996R_tibia, origin xyz=-0.07467046999999999 -0.07467047000000002 0.0 rpy=-3.141592653589793 7.056345106627914e-30 1.5777218104420236e-30
- added joint leg_leg_2_MG996R_femur: type fixed, parent leg_2_MG996R_femur, child leg_2_femur, origin xyz=-0.006505382386916309 0.03106621 -0.013930003589374955 rpy=-5.248374545410663e-16 0.7853981633974433 3.141592653589793
- added joint leg_leg_2_femur_MG996R: type fixed, parent leg_2_femur, child leg_2_MG996R_tibia, origin xyz=-0.10559999999999999 0.0 0.0 rpy=-3.141592653589793 -1.135287644644703e-30 -1.5777218104420236e-30
- added joint leg_leg_3_MG996R_femur: type fixed, parent leg_3_MG996R_femur, child leg_3_femur, origin xyz=0.012020419300373853 0.032184819999999996 0.004595798097915056 rpy=-4.693263033098109e-16 0.7853981633974433 -3.141592653589793
- added joint leg_leg_3_femur_MG996R: type fixed, parent leg_3_femur, child leg_3_MG996R_tibia, origin xyz=-0.07467047000000002 0.07467047000000002 0.0 rpy=3.141592653589793 9.509787901705745e-30 -1.5777218104420236e-30
- added joint leg_leg_4_MG996R_femur: type fixed, parent leg_4_MG996R_femur, child leg_4_femur, origin xyz=0.026470415074497888 -0.01174944 0.019045793872038887 rpy=-4.693263033098162e-16 0.7853981633974433 3.141592653589793
- added joint leg_leg_4_femur_MG996R: type fixed, parent leg_4_femur, child leg_4_MG996R_tibia, origin xyz=0.04030507999999999 0.040305080000000014 0.0 rpy=-3.141592653589793 1.4056744540022418e-29 -3.1554436208840472e-30
- added joint leg_leg_5_MG996R_femur: type fixed, parent leg_5_MG996R_femur, child leg_5_femur, origin xyz=0.013930003589375026 -0.031066209999999997 0.006505382386916168 rpy=-5.248374545410629e-16 0.7853981633974433 3.141592653589793
- added joint leg_leg_5_femur_MG996R: type fixed, parent leg_5_femur, child leg_5_MG996R_tibia, origin xyz=0.056999999999999995 0.0 0.0 rpy=3.141592653589793 2.505999984693438e-31 1.5777218104420236e-30
- added joint leg_leg_6_MG996R_femur: type fixed, parent leg_6_MG996R_femur, child leg_6_femur, origin xyz=-0.004595798097915136 -0.032184819999999996 -0.012020419300373826 rpy=-4.693263033098209e-16 0.7853981633974433 -3.141592653589793
- added joint leg_leg_6_femur_MG996R: type fixed, parent leg_6_femur, child leg_6_MG996R_tibia, origin xyz=0.04030507999999999 -0.04030507999999998 0.0 rpy=3.141592653589793 1.1441314436637283e-29 -1.5777218104420233e-30

Commit message: Slight offset on leg 4 tibia joint

File: hexapod.urdf (robot description, URDF)
Before this commit: robot hexapod, 37 links, 36 joints
Joints:
- joint leg_4_tibia: axis -0.707107 0.707107 4.337944936001927e-29 -> -0.707107 0.707107 4.1148213087586793e-29; origin xyz=0.048377570000000016 -0.001049199999999999 -0.005250000000000001 rpy=3.141592653589793 -3.392272815550781e-28 -4.592132580746781e-86 -> xyz=0.04668052000000001 -0.002746249999999968 -0.005250000000000001 rpy=-3.141592653589793 -3.392272815550781e-28 -1.5777218104420236e-30
