Commit message: Regenerated URDF to use actual parts

File: hexapod.urdf (robot description, URDF)
Before this commit: robot hexapod, 37 links, 36 joints
Links:
- removed link leg_1_MG996R_coxa
- removed link leg_1_MG996R_femur
- removed link leg_1_MG996R_tibia
- removed link leg_1_coxa
- removed link leg_2_MG996R_coxa
- removed link leg_2_MG996R_femur
- removed link leg_2_MG996R_tibia
- removed link leg_2_coxa
- removed link leg_3_MG996R_coxa
- removed link leg_3_MG996R_femur
- removed link leg_3_MG996R_tibia
- removed link leg_3_coxa
- removed link leg_4_MG996R_coxa
- removed link leg_4_MG996R_femur
- removed link leg_4_MG996R_tibia
- removed link leg_4_coxa
- removed link leg_5_MG996R_coxa
- removed link leg_5_MG996R_femur
- removed link leg_5_MG996R_tibia
- removed link leg_5_coxa
- removed link leg_6_MG996R_coxa
- removed link leg_6_MG996R_femur
- removed link leg_6_MG996R_tibia
- added link leg_1_coxa_bracket, mass 0.12359002664125897; collision mesh filename=CAD/motor_bracket.stl scale=0.001 0.001 0.001; visual mesh filename=CAD/motor_bracket.stl scale=0.001 0.001 0.001
- added link leg_1_coxa_motor, mass 0.20795327871559424; collision mesh filename=CAD/MG996R.stl scale=0.001 0.001 0.001; visual mesh filename=CAD/MG996R.stl scale=0.001 0.001 0.001
- added link leg_1_femur_bracket, mass 0.12359002664125897; collision mesh filename=CAD/motor_bracket.stl scale=0.001 0.001 0.001; visual mesh filename=CAD/motor_bracket.stl scale=0.001 0.001 0.001
- added link leg_1_femur_motor, mass 0.20795327871559424; collision mesh filename=CAD/MG996R.stl scale=0.001 0.001 0.001; visual mesh filename=CAD/MG996R.stl scale=0.001 0.001 0.001
- added link leg_1_tibia_bracket, mass 0.12359002664125897; collision mesh filename=CAD/motor_bracket.stl scale=0.001 0.001 0.001; visual mesh filename=CAD/motor_bracket.stl scale=0.001 0.001 0.001
- added link leg_1_tibia_motor, mass 0.20795327871559424; collision mesh filename=CAD/MG996R.stl scale=0.001 0.001 0.001; visual mesh filename=CAD/MG996R.stl scale=0.001 0.001 0.001
- added link leg_2_coxa_bracket, mass 0.12359002664125897; collision mesh filename=CAD/motor_bracket.stl scale=0.001 0.001 0.001; visual mesh filename=CAD/motor_bracket.stl scale=0.001 0.001 0.001
- added link leg_2_coxa_motor, mass 0.20795327871559424; collision mesh filename=CAD/MG996R.stl scale=0.001 0.001 0.001; visual mesh filename=CAD/MG996R.stl scale=0.001 0.001 0.001
- added link leg_2_femur_bracket, mass 0.12359002664125897; collision mesh filename=CAD/motor_bracket.stl scale=0.001 0.001 0.001; visual mesh filename=CAD/motor_bracket.stl scale=0.001 0.001 0.001
- added link leg_2_femur_motor, mass 0.20795327871559424; collision mesh filename=CAD/MG996R.stl scale=0.001 0.001 0.001; visual mesh filename=CAD/MG996R.stl scale=0.001 0.001 0.001
- added link leg_2_tibia_bracket, mass 0.12359002664125897; collision mesh filename=CAD/motor_bracket.stl scale=0.001 0.001 0.001; visual mesh filename=CAD/motor_bracket.stl scale=0.001 0.001 0.001
- added link leg_2_tibia_motor, mass 0.20795327871559424; collision mesh filename=CAD/MG996R.stl scale=0.001 0.001 0.001; visual mesh filename=CAD/MG996R.stl scale=0.001 0.001 0.001
- added link leg_3_coxa_bracket, mass 0.12359002664125897; collision mesh filename=CAD/motor_bracket.stl scale=0.001 0.001 0.001; visual mesh filename=CAD/motor_bracket.stl scale=0.001 0.001 0.001
- added link leg_3_coxa_motor, mass 0.20795327871559424; collision mesh filename=CAD/MG996R.stl scale=0.001 0.001 0.001; visual mesh filename=CAD/MG996R.stl scale=0.001 0.001 0.001
- added link leg_3_femur_bracket, mass 0.12359002664125897; collision mesh filename=CAD/motor_bracket.stl scale=0.001 0.001 0.001; visual mesh filename=CAD/motor_bracket.stl scale=0.001 0.001 0.001
- added link leg_3_femur_motor, mass 0.20795327871559424; collision mesh filename=CAD/MG996R.stl scale=0.001 0.001 0.001; visual mesh filename=CAD/MG996R.stl scale=0.001 0.001 0.001
- added link leg_3_tibia_bracket, mass 0.12359002664125897; collision mesh filename=CAD/motor_bracket.stl scale=0.001 0.001 0.001; visual mesh filename=CAD/motor_bracket.stl scale=0.001 0.001 0.001
- added link leg_3_tibia_motor, mass 0.20795327871559424; collision mesh filename=CAD/MG996R.stl scale=0.001 0.001 0.001; visual mesh filename=CAD/MG996R.stl scale=0.001 0.001 0.001
- added link leg_4_coxa_bracket, mass 0.12359002664125897; collision mesh filename=CAD/motor_bracket.stl scale=0.001 0.001 0.001; visual mesh filename=CAD/motor_bracket.stl scale=0.001 0.001 0.001
- added link leg_4_coxa_motor, mass 0.20795327871559424; collision mesh filename=CAD/MG996R.stl scale=0.001 0.001 0.001; visual mesh filename=CAD/MG996R.stl scale=0.001 0.001 0.001
- added link leg_4_femur_bracket, mass 0.12359002664125897; collision mesh filename=CAD/motor_bracket.stl scale=0.001 0.001 0.001; visual mesh filename=CAD/motor_bracket.stl scale=0.001 0.001 0.001
- added link leg_4_femur_motor, mass 0.20795327871559424; collision mesh filename=CAD/MG996R.stl scale=0.001 0.001 0.001; visual mesh filename=CAD/MG996R.stl scale=0.001 0.001 0.001
- added link leg_4_tibia_bracket, mass 0.12359002664125897; collision mesh filename=CAD/motor_bracket.stl scale=0.001 0.001 0.001; visual mesh filename=CAD/motor_bracket.stl scale=0.001 0.001 0.001
- added link leg_4_tibia_motor, mass 0.20795327871559424; collision mesh filename=CAD/MG996R.stl scale=0.001 0.001 0.001; visual mesh filename=CAD/MG996R.stl scale=0.001 0.001 0.001
- added link leg_5_coxa_bracket, mass 0.12359002664125897; collision mesh filename=CAD/motor_bracket.stl scale=0.001 0.001 0.001; visual mesh filename=CAD/motor_bracket.stl scale=0.001 0.001 0.001
- added link leg_5_coxa_motor, mass 0.20795327871559424; collision mesh filename=CAD/MG996R.stl scale=0.001 0.001 0.001; visual mesh filename=CAD/MG996R.stl scale=0.001 0.001 0.001
- added link leg_5_femur_bracket, mass 0.12359002664125897; collision mesh filename=CAD/motor_bracket.stl scale=0.001 0.001 0.001; visual mesh filename=CAD/motor_bracket.stl scale=0.001 0.001 0.001
- added link leg_5_femur_motor, mass 0.20795327871559424; collision mesh filename=CAD/MG996R.stl scale=0.001 0.001 0.001; visual mesh filename=CAD/MG996R.stl scale=0.001 0.001 0.001
- added link leg_5_tibia_bracket, mass 0.12359002664125897; collision mesh filename=CAD/motor_bracket.stl scale=0.001 0.001 0.001; visual mesh filename=CAD/motor_bracket.stl scale=0.001 0.001 0.001
- added link leg_5_tibia_motor, mass 0.20795327871559424; collision mesh filename=CAD/MG996R.stl scale=0.001 0.001 0.001; visual mesh filename=CAD/MG996R.stl scale=0.001 0.001 0.001
- added link leg_6_coxa_bracket, mass 0.12359002664125897; collision mesh filename=CAD/motor_bracket.stl scale=0.001 0.001 0.001; visual mesh filename=CAD/motor_bracket.stl scale=0.001 0.001 0.001
- added link leg_6_femur_bracket, mass 0.12359002664125897; collision mesh filename=CAD/motor_bracket.stl scale=0.001 0.001 0.001; visual mesh filename=CAD/motor_bracket.stl scale=0.001 0.001 0.001
- added link leg_6_femur_motor, mass 0.20795327871559424; collision mesh filename=CAD/MG996R.stl scale=0.001 0.001 0.001; visual mesh filename=CAD/MG996R.stl scale=0.001 0.001 0.001
- added link leg_6_tibia_bracket, mass 0.12359002664125897; collision mesh filename=CAD/motor_bracket.stl scale=0.001 0.001 0.001; visual mesh filename=CAD/motor_bracket.stl scale=0.001 0.001 0.001
- added link leg_6_tibia_motor, mass 0.20795327871559424; collision mesh filename=CAD/MG996R.stl scale=0.001 0.001 0.001; visual mesh filename=CAD/MG996R.stl scale=0.001 0.001 0.001
- link leg_1_tibia: mass 0.2763071087572843 -> 0.1636969553862354
- link leg_2_tibia: mass 0.2763071087572843 -> 0.1636969553862354
- link leg_3_tibia: mass 0.2763071087572843 -> 0.1636969553862354
- link leg_4_tibia: mass 0.2763071087572843 -> 0.1636969553862354
- link leg_5_tibia: mass 0.2763071087572843 -> 0.1636969553862354
- link leg_6_coxa: mass 0.23210805328252054 -> 0.20795327871559424; geometry collision mesh filename=CAD/leg_6_coxa.stl scale=0.001 0.001 0.001; visual mesh filename=CAD/leg_6_coxa.stl scale=0.001 0.001 0.001
- link leg_6_tibia: mass 0.2763071087572843 -> 0.1636969553862354
Joints:
- removed joint base_leg_1
- removed joint base_leg_2
- removed joint base_leg_3
- removed joint base_leg_4
- removed joint base_leg_5
- removed joint base_leg_6
- removed joint leg_1_coxa
- removed joint leg_1_femur
- removed joint leg_1_tibia
- removed joint leg_2_coxa
- removed joint leg_2_femur
- removed joint leg_2_tibia
- removed joint leg_3_coxa
- removed joint leg_3_femur
- removed joint leg_3_tibia
- removed joint leg_4_coxa
- removed joint leg_4_femur
- removed joint leg_4_tibia
- removed joint leg_5_coxa
- removed joint leg_5_femur
- removed joint leg_5_tibia
- removed joint leg_6_coxa
- removed joint leg_6_femur
- removed joint leg_6_tibia
- removed joint leg_leg_1_MG996R_femur
- removed joint leg_leg_1_femur_MG996R
- removed joint leg_leg_2_MG996R_femur
- removed joint leg_leg_2_femur_MG996R
- removed joint leg_leg_3_MG996R_femur
- removed joint leg_leg_3_femur_MG996R
- removed joint leg_leg_4_MG996R_femur
- removed joint leg_leg_4_femur_MG996R
- removed joint leg_leg_5_MG996R_femur
- removed joint leg_leg_5_femur_MG996R
- removed joint leg_leg_6_MG996R_femur
- removed joint leg_leg_6_femur_MG996R
- added joint base_body_leg_1_coxa_motor: type fixed, parent base, child leg_1_coxa_motor, origin xyz=0.03687243816741341 0.054812817597825615 -3.6152416083012894e-09 rpy=-6.556553535888259e-16 -1.883898413669496e-21 -3.14159265358979
- added joint base_body_leg_2_coxa_motor: type fixed, parent base, child leg_2_coxa_motor, origin xyz=0.0371349981674136 -0.005250002402174338 -3.6152416527102107e-09 rpy=-6.556553535888259e-16 -1.883898413669496e-21 -3.14159265358979
- added joint base_body_leg_3_coxa_motor: type fixed, parent base, child leg_3_coxa_motor, origin xyz=0.029447818167413774 -0.062237432402174345 -3.6152416882373475e-09 rpy=-6.556553535888259e-16 -1.883898413669496e-21 -3.14159265358979
- added joint base_body_leg_4_coxa_motor: type fixed, parent base, child leg_4_coxa_motor, origin xyz=-0.03687244183258621 -0.05481281240217456 -3.615241679355563e-09 rpy=-6.556553535888259e-16 -1.883898413669496e-21 -3.14159265358979
- added joint base_body_leg_5_coxa_motor: type fixed, parent base, child leg_5_coxa_motor, origin xyz=-0.03713500183258638 0.0052499975978254195 -3.6152416438284263e-09 rpy=-6.556553535888259e-16 -1.883898413669496e-21 -3.14159265358979
- added joint base_body_leg_6_coxa_motor: type fixed, parent base, child leg_6_coxa, origin xyz=-0.02944781183258657 0.0622374375978254 -3.6152416083012894e-09 rpy=-6.556553535888259e-16 -1.883898413669496e-21 -3.14159265358979
- added joint leg_1_coxa_bracket_leg_1_coxa_bracket_femur_bracket: type fixed, parent leg_1_coxa_bracket, child leg_1_femur_bracket, origin xyz=-0.027577160000000003 -0.020506100000000006 -0.016499999999999994 rpy=-2.8108466990367964e-32 -2.465190328815662e-32 -1.159930852145538e-30
- added joint leg_1_coxa_motor_leg_1_coxa: type continuous, parent leg_1_coxa_motor, child leg_1_coxa_bracket, origin xyz=-0.02100107 -0.02842569000000001 0.03106622 rpy=-9.860761315262648e-32 3.76158192263132e-37 1.5543625399441258e-30, axis 0.0 9.860761315262648e-32 -1.0
- added joint leg_1_femur_bracket_leg_1_femur: type continuous, parent leg_1_femur_bracket, child leg_1_femur_motor, origin xyz=-0.035708899999999995 -0.012374369999999999 -0.005 rpy=4.440892098500626e-16 -1.5707963267948966 0, axis 8.033749522571572e-32 0.7071070000000004 0.7071069999999996
- added joint leg_1_femur_leg_1_femur_tibia_motor: type fixed, parent leg_1_femur, child leg_1_tibia_motor, origin xyz=-0.07467048 -0.07467048000000003 0.0 rpy=3.141592653589793 1.5446002659865263e-32 1.2325951644078318e-32
- added joint leg_1_femur_motor_leg_1_femur_motor_femur: type fixed, parent leg_1_femur_motor, child leg_1_femur, origin xyz=0.005249999999999995 -0.01174942999999999 -0.03218482999999999 rpy=-2.4651903288158053e-32 1.5707963267948961 0
- added joint leg_1_tibia_bracket_leg_1_tibia_bracket_tibia: type fixed, parent leg_1_tibia_bracket, child leg_1_tibia, origin xyz=-0.0053032999999999934 -0.042779960000000006 0.005 rpy=8.628166150854817e-32 -1.2833170489735542e-31 -6.162975822039156e-32
- added joint leg_1_tibia_motor_leg_1_tibia: type continuous, parent leg_1_tibia_motor, child leg_1_tibia_bracket, origin xyz=-0.01174944 -0.032184819999999996 0.005249999999999986 rpy=-3.141592653589793 -2.616422446273694e-31 6.162975822039157e-32, axis 0.707107 -0.7071069999999999 1.7788994558731144e-30
- added joint leg_2_coxa_bracket_leg_2_coxa_bracket_femur_bracket: type fixed, parent leg_2_coxa_bracket, child leg_2_femur_bracket, origin xyz=-0.034 0.005 -0.01649999999999999 rpy=-1.5865212034703782e-31 1.1551963198647533e-62 1.1715082466063972e-31
- added joint leg_2_coxa_motor_leg_2_coxa: type continuous, parent leg_2_coxa_motor, child leg_2_coxa_bracket, origin xyz=-0.034949999999999995 -0.005249999999999986 0.03106622 rpy=9.86076131526265e-32 3.76158192263132e-37 4.74496089443201e-31, axis 0.0 -9.860761315262648e-32 -0.9999999999999999
- added joint leg_2_femur_bracket_leg_2_femur: type continuous, parent leg_2_femur_bracket, child leg_2_femur_motor, origin xyz=-0.033999999999999996 0.016499999999999987 -0.005 rpy=4.440892098500624e-16 -1.5707963267948966 0, axis -1.9721522630525295e-31 1.0 -4.440892098500626e-16
- added joint leg_2_femur_leg_2_femur_tibia_motor: type fixed, parent leg_2_femur, child leg_2_tibia_motor, origin xyz=-0.10560000000000003 -3.552713678800501e-17 0.0 rpy=-3.141592653589793 1.8278101094214132e-31 -1.9721522630525295e-31
- added joint leg_2_femur_motor_leg_2_femur_motor_femur: type fixed, parent leg_2_femur_motor, child leg_2_femur, origin xyz=0.005249999999999995 -0.03106621999999998 -0.014449999999999985 rpy=-1.9721522630525295e-31 1.5707963267948961 0
- added joint leg_2_tibia_bracket_leg_2_tibia_bracket_tibia: type fixed, parent leg_2_tibia_bracket, child leg_2_tibia, origin xyz=-0.03399999999999999 -0.026499999999999985 0.005 rpy=1.97215226305253e-31 -1.4466484721319702e-31 9.860761315262648e-32
- added joint leg_2_tibia_motor_leg_2_tibia: type continuous, parent leg_2_tibia_motor, child leg_2_tibia_bracket, origin xyz=0.014450000000000003 -0.03106621999999998 0.005249999999999995 rpy=3.141592653589793 6.2423205830278e-32 -1.0285368061487781e-63, axis 9.860761315262648e-32 -1.0 0.0
- added joint leg_3_coxa_bracket_leg_3_coxa_bracket_femur_bracket: type fixed, parent leg_3_coxa_bracket, child leg_3_femur_bracket, origin xyz=-0.0205061 0.02757715999999995 -0.016499999999999994 rpy=-1.0087333778760568e-31 -1.9721522630525295e-31 -1.0268577116000727e-30
- added joint leg_3_coxa_motor_leg_3_coxa: type continuous, parent leg_3_coxa_motor, child leg_3_coxa_bracket, origin xyz=-0.028425690000000003 0.021001079999999988 0.03106622 rpy=-9.860761315262648e-32 3.76158192263132e-37 1.3473336895341905e-30, axis 0.0 9.860761315262648e-32 -1.0
- added joint leg_3_femur_bracket_leg_3_femur: type continuous, parent leg_3_femur_bracket, child leg_3_femur_motor, origin xyz=-0.012374369999999999 0.035708890000000014 -0.004999999999999991 rpy=4.440892098500626e-16 -1.5707963267948966 0, axis -5.485808580416637e-31 0.7071069999999997 -0.7071070000000004
- added joint leg_3_femur_leg_3_femur_motor_femur: type fixed, parent leg_3_femur, child leg_3_femur_motor, origin xyz=0.08130000157835046 0.005250003181322987 0.013999998099572046 rpy=1.570796326794896 0.7853981633974517 2.194934138149569e-15
- added joint leg_3_femur_leg_3_femur_tibia_motor: type fixed, parent leg_3_femur, child leg_3_tibia_motor, origin xyz=-0.02430000394655856 0.005250003181322853 0.013999998099572508 rpy=1.570796326794896 0.7853981633974517 2.194934138149569e-15
- added joint leg_3_tibia_bracket_leg_3_tibia_bracket_tibia: type fixed, parent leg_3_tibia_bracket, child leg_3_tibia, origin xyz=-0.04277996 0.0053032999999999934 0.005 rpy=1.9721522630525295e-31 5.9314479861815994e-30 1.1697718569126413e-60
- added joint leg_3_tibia_motor_leg_3_tibia: type continuous, parent leg_3_tibia_motor, child leg_3_tibia_bracket, origin xyz=0.032184819999999996 -0.01174942999999999 0.005249999999999995 rpy=3.141592653589793 4.0080150659657764e-30 0.0, axis -0.707107 -0.7071069999999999 -5.036747943978376e-30
- added joint leg_4_coxa_bracket_leg_4_coxa_bracket_femur_bracket: type fixed, parent leg_4_coxa_bracket, child leg_4_femur_bracket, origin xyz=0.027577160000000003 0.020506089999999946 -0.016499999999999994 rpy=2.549406408329769e-30 -1.9721522630525295e-31 9.271701804161562e-31
- added joint leg_4_coxa_motor_leg_4_coxa: type continuous, parent leg_4_coxa_motor, child leg_4_coxa_bracket, origin xyz=0.021001069999999997 0.028425700000000022 0.03106622 rpy=8.521886419342739e-67 3.76158192263132e-37 -5.327384926175685e-31, axis 0.0 0.0 -1.0
- added joint leg_4_femur_bracket_leg_4_femur: type continuous, parent leg_4_femur_bracket, child leg_4_femur_motor, origin xyz=0.035708890000000014 0.012374369999999999 -0.005 rpy=4.440892098500626e-16 -1.5707963267948966 0, axis 8.07701892512926e-31 -0.7071070000000004 -0.7071069999999997
- added joint leg_4_femur_leg_4_femur_tibia_motor: type fixed, parent leg_4_femur, child leg_4_tibia_motor, origin xyz=0.07467048 0.07467047000000002 0.0 rpy=3.141592653589793 3.952172413649149e-31 3.944304526105059e-31
- added joint leg_4_femur_motor_leg_4_femur_motor_femur: type fixed, parent leg_4_femur_motor, child leg_4_femur, origin xyz=0.005249999999999995 0.011749440000000036 0.032184819999999996 rpy=-1.226136156284215e-44 1.5707963267948961 0
- added joint leg_4_tibia_bracket_leg_4_tibia_bracket_tibia: type fixed, parent leg_4_tibia_bracket, child leg_4_tibia, origin xyz=0.005303300000000029 0.04277996000000002 0.005 rpy=2.2227780068508204e-59 1.19525921236697e-29 3.94430452610506e-31
- added joint leg_4_tibia_motor_leg_4_tibia: type continuous, parent leg_4_tibia_motor, child leg_4_tibia_bracket, origin xyz=0.01174942999999999 0.03218482000000002 0.005249999999999995 rpy=3.141592653589793 9.139245607922579e-30 3.604796781651481e-60, axis -0.707107 0.7071069999999999 -1.4430361871667657e-29
- added joint leg_5_coxa_bracket_leg_5_coxa_bracket_femur_bracket: type fixed, parent leg_5_coxa_bracket, child leg_5_femur_bracket, origin xyz=0.034 -0.005 -0.016499999999999994 rpy=3.944271066555727e-31 1.9721522630525295e-31 4.9933280800949095e-31
- added joint leg_5_coxa_motor_leg_5_coxa: type continuous, parent leg_5_coxa_motor, child leg_5_coxa_bracket, origin xyz=0.034949999999999995 0.005250000000000021 0.03106622 rpy=-3.944304526105059e-31 -1.9721485014706069e-31 9.231410609434975e-32, axis -1.9721522630525295e-31 3.944304526105059e-31 -1.0
- added joint leg_5_femur_bracket_leg_5_femur: type continuous, parent leg_5_femur_bracket, child leg_5_femur_motor, origin xyz=0.034 -0.01650000000000002 -0.005 rpy=4.440892098500624e-16 -1.5707963267948966 0, axis 2.465190328815662e-32 -1.0 4.440892098500626e-16
- added joint leg_5_femur_leg_5_femur_tibia_motor: type fixed, parent leg_5_femur, child leg_5_tibia_motor, origin xyz=0.10559999999999997 -3.552713678800501e-17 0.0 rpy=3.141592653589793 7.009300602024574e-32 -2.4651903288156624e-32
- added joint leg_5_femur_motor_leg_5_femur_motor_femur: type fixed, parent leg_5_femur_motor, child leg_5_femur, origin xyz=0.005249999999999995 0.031066210000000007 0.014449999999999985 rpy=7.642090019328554e-31 1.5707963267948961 0
- added joint leg_5_tibia_bracket_leg_5_tibia_bracket_tibia: type fixed, parent leg_5_tibia_bracket, child leg_5_tibia, origin xyz=0.033999999999999954 0.026499999999999985 0.005 rpy=1.4017973344692734e-61 -1.3982310497502855e-31 7.888609052210118e-31
- added joint leg_5_tibia_motor_leg_5_tibia: type continuous, parent leg_5_tibia_motor, child leg_5_tibia_bracket, origin xyz=-0.014449999999999968 0.031066210000000007 0.005249999999999995 rpy=3.141592653589793 -1.5263675252030436e-31 0.0, axis 0.0 0.9999999999999999 3.944304526105059e-31
- added joint leg_6_coxa_bracket_leg_6_coxa_bracket_femur_bracket: type fixed, parent leg_6_coxa_bracket, child leg_6_femur_bracket, origin xyz=0.020506090000000015 -0.027577169999999995 -0.016500000000000004 rpy=4.299763345216673e-31 1.97215226305253e-31 6.034920170673757e-31
- added joint leg_6_coxa_leg_6_coxa: type continuous, parent leg_6_coxa, child leg_6_coxa_bracket, origin xyz=0.028425699999999995 -0.021001070000000014 0.03346622 rpy=-1.97215226305253e-31 -1.9721485014706069e-31 -1.1845102963535013e-32, axis -1.9721522630525295e-31 1.9721522630525295e-31 -0.9999999999999999
- added joint leg_6_femur_bracket_leg_6_femur: type continuous, parent leg_6_femur_bracket, child leg_6_femur_motor, origin xyz=0.012374369999999999 -0.035708890000000014 -0.005 rpy=4.440892098500624e-16 -1.5707963267948966 0, axis -4.574311772530478e-32 -0.7071069999999996 0.7071070000000003
- added joint leg_6_femur_leg_6_femur_tibia_motor: type fixed, parent leg_6_femur, child leg_6_tibia_motor, origin xyz=0.07467047000000003 -0.07467048000000003 8.881784197001253e-18 rpy=3.141592653589793 -2.264625944649728e-32 2.4651903288156613e-32
- added joint leg_6_femur_motor_leg_6_femur_motor_femur: type fixed, parent leg_6_femur_motor, child leg_6_femur, origin xyz=0.0052500000000000125 0.03218483000000001 -0.01174944 rpy=4.314083075426797e-32 1.5707963267948961 0
- added joint leg_6_tibia_bracket_leg_6_tibia_bracket_tibia: type fixed, parent leg_6_tibia_bracket, child leg_6_tibia, origin xyz=0.04277996000000002 -0.005303300000000002 0.004999999999999991 rpy=-1.1093356479670479e-31 -9.280960075532134e-31 2.465190328815662e-32
- added joint leg_6_tibia_motor_leg_6_tibia: type continuous, parent leg_6_tibia_motor, child leg_6_tibia_bracket, origin xyz=-0.03218482000000002 0.01174944 0.005250000000000004 rpy=-3.141592653589793 -1.187439434814482e-30 1.355854680848614e-31, axis 0.7071070000000002 0.707107 7.512391405886096e-30

Commit message: Incorrect mesh for leg 6 coxa

File: hexapod.urdf (robot description, URDF)
Before this commit: robot Hexapod, 49 links, 48 joints
Links:
- link leg_6_coxa: geometry collision mesh filename=CAD/coxa.stl scale=0.001 0.001 0.001; visual mesh filename=CAD/coxa.stl scale=0.001 0.001 0.001

Commit message: Incorrect mesh for leg 6 coxa

File: hexapod.urdf (robot description, URDF)
Before this commit: robot Hexapod, 49 links, 48 joints
Links:
- removed link leg_6_coxa
- added link leg_6_coxa_motor, mass 0.20795327871559424; collision mesh filename=CAD/MG996R.stl scale=0.001 0.001 0.001; visual mesh filename=CAD/MG996R.stl scale=0.001 0.001 0.001
Joints:
- joint base_body_leg_6_coxa_motor: child leg_6_coxa -> leg_6_coxa_motor
- joint leg_6_coxa_leg_6_coxa: parent leg_6_coxa -> leg_6_coxa_motor
