Commit message: Corrupted joint leg 3

File: hexapod.urdf (robot description, URDF)
Before this commit: robot Hexapod, 49 links, 48 joints
Links:
- link leg_3_coxa_bracket: geometry collision mesh filename=meshes/motor_bracket.stl scale=0.001 0.001 0.001; visual mesh filename=meshes/motor_bracket.stl scale=0.001 0.001 0.001
- link leg_3_coxa_motor: geometry collision mesh filename=meshes/MG996R.stl scale=0.001 0.001 0.001; visual mesh filename=meshes/MG996R.stl scale=0.001 0.001 0.001
- link leg_3_femur: geometry collision mesh filename=meshes/femur.stl scale=0.001 0.001 0.001; visual mesh filename=meshes/femur.stl scale=0.001 0.001 0.001
- link leg_3_femur_bracket: geometry collision mesh filename=meshes/motor_bracket.stl scale=0.001 0.001 0.001; visual mesh filename=meshes/motor_bracket.stl scale=0.001 0.001 0.001
- link leg_3_femur_motor: geometry collision mesh filename=meshes/MG996R.stl scale=0.001 0.001 0.001; visual mesh filename=meshes/MG996R.stl scale=0.001 0.001 0.001
- link leg_3_tibia: geometry collision mesh filename=meshes/tibia.stl scale=0.001 0.001 0.001; visual mesh filename=meshes/tibia.stl scale=0.001 0.001 0.001
- link leg_3_tibia_bracket: geometry collision mesh filename=meshes/motor_bracket.stl scale=0.001 0.001 0.001; visual mesh filename=meshes/motor_bracket.stl scale=0.001 0.001 0.001
- link leg_3_tibia_motor: geometry collision mesh filename=meshes/MG996R.stl scale=0.001 0.001 0.001; visual mesh filename=meshes/MG996R.stl scale=0.001 0.001 0.001
Joints:
- removed joint leg_3_femur_leg_3_femur_motor_femur
- removed joint leg_6_coxa_leg_6_coxa
- added joint leg_3_femur_motor_leg_3_femur_motor_femur: type fixed, parent leg_3_femur_motor, child leg_3_femur, origin xyz=0.005249999999999995 -0.03218482000000002 0.011749430000000017 rpy=-3.944304526105096e-31 1.5707963267948961 0
- added joint leg_6_coxa_leg_6_coxa_motor: type continuous, parent leg_6_coxa_motor, child leg_6_coxa_bracket, origin xyz=0.028425699999999995 -0.021001070000000014 0.03346622 rpy=-1.97215226305253e-31 -1.9721485014706069e-31 -1.1845102963535013e-32, axis -1.9721522630525295e-31 1.9721522630525295e-31 -0.9999999999999999
- joint leg_3_femur_leg_3_femur_tibia_motor: origin xyz=-0.02430000394655856 0.005250003181322853 0.013999998099572508 rpy=1.570796326794896 0.7853981633974517 2.194934138149569e-15 -> xyz=-0.07467048 0.07467048000000005 0.0 rpy=3.141592653589793 2.9749109199195536e-31 -3.944304526105059e-31
- joint leg_3_tibia_bracket_leg_3_tibia_bracket_tibia: origin xyz=-0.04277996 0.0053032999999999934 0.005 rpy=1.9721522630525295e-31 5.9314479861815994e-30 1.1697718569126413e-60 -> xyz=-0.04277996 0.0053032999999999934 0.005 rpy=5.916456789157587e-31 5.143330097529235e-30 2.433999741754704e-61
- joint leg_3_tibia_motor_leg_3_tibia: axis -0.707107 -0.7071069999999999 -5.036747943978376e-30 -> -0.707107 -0.7071070000000002 -4.9975677246065126e-30; origin xyz=0.032184819999999996 -0.01174942999999999 0.005249999999999995 rpy=3.141592653589793 4.0080150659657764e-30 0.0 -> xyz=0.032184819999999996 -0.01174942999999999 0.005249999999999995 rpy=3.141592653589793 2.5209203703305588e-30 -1.9721522630525295e-31

Commit message: Renamed joints

File: hexapod.urdf (robot description, URDF)
Before this commit: robot Hexapod, 49 links, 48 joints
Joints:
- removed joint leg_1_coxa_motor_leg_1_coxa
- removed joint leg_1_femur_bracket_leg_1_femur
- removed joint leg_1_tibia_motor_leg_1_tibia
- removed joint leg_2_coxa_motor_leg_2_coxa
- removed joint leg_2_femur_bracket_leg_2_femur
- removed joint leg_2_tibia_motor_leg_2_tibia
- removed joint leg_3_coxa_motor_leg_3_coxa
- removed joint leg_3_femur_bracket_leg_3_femur
- removed joint leg_3_tibia_motor_leg_3_tibia
- removed joint leg_4_coxa_motor_leg_4_coxa
- removed joint leg_4_femur_bracket_leg_4_femur
- removed joint leg_4_tibia_motor_leg_4_tibia
- removed joint leg_5_coxa_motor_leg_5_coxa
- removed joint leg_5_femur_bracket_leg_5_femur
- removed joint leg_5_tibia_motor_leg_5_tibia
- removed joint leg_6_femur_bracket_leg_6_femur
- removed joint leg_6_tibia_motor_leg_6_tibia
- added joint leg_1_coxa: type continuous, parent leg_1_coxa_motor, child leg_1_coxa_bracket, origin xyz=-0.02100107 -0.02842569000000001 0.03106622 rpy=-9.860761315262648e-32 3.76158192263132e-37 1.5543625399441258e-30, axis 0.0 9.860761315262648e-32 -1.0
- added joint leg_1_femur: type continuous, parent leg_1_femur_bracket, child leg_1_femur_motor, origin xyz=-0.035708899999999995 -0.012374369999999999 -0.005 rpy=4.440892098500626e-16 -1.5707963267948966 0, axis 8.033749522571572e-32 0.7071070000000004 0.7071069999999996
- added joint leg_1_tibia: type continuous, parent leg_1_tibia_motor, child leg_1_tibia_bracket, origin xyz=-0.01174944 -0.032184819999999996 0.005249999999999986 rpy=-3.141592653589793 -2.616422446273694e-31 6.162975822039157e-32, axis 0.707107 -0.7071069999999999 1.7788994558731144e-30
- added joint leg_2_coxa: type continuous, parent leg_2_coxa_motor, child leg_2_coxa_bracket, origin xyz=-0.034949999999999995 -0.005249999999999986 0.03106622 rpy=9.86076131526265e-32 3.76158192263132e-37 4.74496089443201e-31, axis 0.0 -9.860761315262648e-32 -0.9999999999999999
- added joint leg_2_femur: type continuous, parent leg_2_femur_bracket, child leg_2_femur_motor, origin xyz=-0.033999999999999996 0.016499999999999987 -0.005 rpy=4.440892098500624e-16 -1.5707963267948966 0, axis -1.9721522630525295e-31 1.0 -4.440892098500626e-16
- added joint leg_2_tibia: type continuous, parent leg_2_tibia_motor, child leg_2_tibia_bracket, origin xyz=0.014450000000000003 -0.03106621999999998 0.005249999999999995 rpy=3.141592653589793 6.2423205830278e-32 -1.0285368061487781e-63, axis 9.860761315262648e-32 -1.0 0.0
- added joint leg_3_coxa: type continuous, parent leg_3_coxa_motor, child leg_3_coxa_bracket, origin xyz=-0.028425690000000003 0.021001079999999988 0.03106622 rpy=-9.860761315262648e-32 3.76158192263132e-37 1.3473336895341905e-30, axis 0.0 9.860761315262648e-32 -1.0
- added joint leg_3_femur: type continuous, parent leg_3_femur_bracket, child leg_3_femur_motor, origin xyz=-0.012374369999999999 0.035708890000000014 -0.004999999999999991 rpy=4.440892098500626e-16 -1.5707963267948966 0, axis -5.485808580416637e-31 0.7071069999999997 -0.7071070000000004
- added joint leg_3_tibia: type continuous, parent leg_3_tibia_motor, child leg_3_tibia_bracket, origin xyz=0.032184819999999996 -0.01174942999999999 0.005249999999999995 rpy=3.141592653589793 2.5209203703305588e-30 -1.9721522630525295e-31, axis -0.707107 -0.7071070000000002 -4.9975677246065126e-30
- added joint leg_4_coxa: type continuous, parent leg_4_coxa_motor, child leg_4_coxa_bracket, origin xyz=0.021001069999999997 0.028425700000000022 0.03106622 rpy=8.521886419342739e-67 3.76158192263132e-37 -5.327384926175685e-31, axis 0.0 0.0 -1.0
- added joint leg_4_femur: type continuous, parent leg_4_femur_bracket, child leg_4_femur_motor, origin xyz=0.035708890000000014 0.012374369999999999 -0.005 rpy=4.440892098500626e-16 -1.5707963267948966 0, axis 8.07701892512926e-31 -0.7071070000000004 -0.7071069999999997
- added joint leg_4_tibia: type continuous, parent leg_4_tibia_motor, child leg_4_tibia_bracket, origin xyz=0.01174942999999999 0.03218482000000002 0.005249999999999995 rpy=3.141592653589793 9.139245607922579e-30 3.604796781651481e-60, axis -0.707107 0.7071069999999999 -1.4430361871667657e-29
- added joint leg_5_coxa: type continuous, parent leg_5_coxa_motor, child leg_5_coxa_bracket, origin xyz=0.034949999999999995 0.005250000000000021 0.03106622 rpy=-3.944304526105059e-31 -1.9721485014706069e-31 9.231410609434975e-32, axis -1.9721522630525295e-31 3.944304526105059e-31 -1.0
- added joint leg_5_femur: type continuous, parent leg_5_femur_bracket, child leg_5_femur_motor, origin xyz=0.034 -0.01650000000000002 -0.005 rpy=4.440892098500624e-16 -1.5707963267948966 0, axis 2.465190328815662e-32 -1.0 4.440892098500626e-16
- added joint leg_5_tibia: type continuous, parent leg_5_tibia_motor, child leg_5_tibia_bracket, origin xyz=-0.014449999999999968 0.031066210000000007 0.005249999999999995 rpy=3.141592653589793 -1.5263675252030436e-31 0.0, axis 0.0 0.9999999999999999 3.944304526105059e-31
- added joint leg_6_femur: type continuous, parent leg_6_femur_bracket, child leg_6_femur_motor, origin xyz=0.012374369999999999 -0.035708890000000014 -0.005 rpy=4.440892098500624e-16 -1.5707963267948966 0, axis -4.574311772530478e-32 -0.7071069999999996 0.7071070000000003
- added joint leg_6_tibia: type continuous, parent leg_6_tibia_motor, child leg_6_tibia_bracket, origin xyz=-0.03218482000000002 0.01174944 0.005250000000000004 rpy=-3.141592653589793 -1.187439434814482e-30 1.355854680848614e-31, axis 0.7071070000000002 0.707107 7.512391405886096e-30

Commit message: Typo in joint 6 coxa name

File: hexapod.urdf (robot description, URDF)
Before this commit: robot Hexapod, 49 links, 48 joints
Joints:
- removed joint leg_6_coxa_leg_6_coxa_motor
- added joint leg_6_coxa: type continuous, parent leg_6_coxa_motor, child leg_6_coxa_bracket, origin xyz=0.028425699999999995 -0.021001070000000014 0.03346622 rpy=-1.97215226305253e-31 -1.9721485014706069e-31 -1.1845102963535013e-32, axis -1.9721522630525295e-31 1.9721522630525295e-31 -0.9999999999999999

Commit message: Added electronics and battery

File: hexapod.urdf (robot description, URDF)
Before this commit: robot Hexapod, 49 links, 48 joints
Links:
- added link battery, mass 1.3563652746505896; collision mesh filename=CAD/battery.stl scale=0.001 0.001 0.001; visual mesh filename=CAD/battery.stl scale=0.001 0.001 0.001
- added link electronics, mass 0.32180259543495077; collision mesh filename=CAD/electronics.stl scale=0.001 0.001 0.001; visual mesh filename=CAD/electronics.stl scale=0.001 0.001 0.001
Joints:
- added joint base_battery: type fixed, parent base, child battery, origin xyz=-1.8325863981871748e-09 -2.4021744593483163e-09 -3.6152416438284263e-09 rpy=3.1415926535897927 -1.883898413669496e-21 -3.14159265358979
- added joint base_electronics: type fixed, parent base, child electronics, origin xyz=-0.03263500183258655 0.057999997597825405 0.013999996384758396 rpy=3.1415926535897927 -1.883898413669496e-21 -3.14159265358979

Commit message: Fixed old mesh path

File: hexapod.urdf (robot description, URDF)
Before this commit: robot Hexapod, 51 links, 50 joints
Links:
- link leg_3_coxa_bracket: geometry collision mesh filename=CAD/motor_bracket.stl scale=0.001 0.001 0.001; visual mesh filename=CAD/motor_bracket.stl scale=0.001 0.001 0.001
- link leg_3_coxa_motor: geometry collision mesh filename=CAD/MG996R.stl scale=0.001 0.001 0.001; visual mesh filename=CAD/MG996R.stl scale=0.001 0.001 0.001
- link leg_3_femur: geometry collision mesh filename=CAD/femur.stl scale=0.001 0.001 0.001; visual mesh filename=CAD/femur.stl scale=0.001 0.001 0.001
- link leg_3_femur_bracket: geometry collision mesh filename=CAD/motor_bracket.stl scale=0.001 0.001 0.001; visual mesh filename=CAD/motor_bracket.stl scale=0.001 0.001 0.001
- link leg_3_femur_motor: geometry collision mesh filename=CAD/MG996R.stl scale=0.001 0.001 0.001; visual mesh filename=CAD/MG996R.stl scale=0.001 0.001 0.001
- link leg_3_tibia: geometry collision mesh filename=CAD/tibia.stl scale=0.001 0.001 0.001; visual mesh filename=CAD/tibia.stl scale=0.001 0.001 0.001
- link leg_3_tibia_bracket: geometry collision mesh filename=CAD/motor_bracket.stl scale=0.001 0.001 0.001; visual mesh filename=CAD/motor_bracket.stl scale=0.001 0.001 0.001
- link leg_3_tibia_motor: geometry collision mesh filename=CAD/MG996R.stl scale=0.001 0.001 0.001; visual mesh filename=CAD/MG996R.stl scale=0.001 0.001 0.001

Commit message: Added electronics

File: hexapod.urdf (robot description, URDF)
Before this commit: robot Hexapod, 70 links, 69 joints
Links:
- removed link base_cover
- removed link mounting_plate
- added link battery_mount, mass 0.1649336841152355; collision mesh filename=CAD/battery_mount.stl scale=0.001 0.001 0.001; visual mesh filename=CAD/battery_mount.stl scale=0.001 0.001 0.001
- added link camera, mass 0.0017238411866737254; collision mesh filename=CAD/camera.stl scale=0.001 0.001 0.001; visual mesh filename=CAD/camera.stl scale=0.001 0.001 0.001
- added link camera_mount, mass 0.001081689709436805; collision mesh filename=CAD/camera_mount.stl scale=0.001 0.001 0.001; visual mesh filename=CAD/camera_mount.stl scale=0.001 0.001 0.001
- added link electronics, mass 0.07571894822352634; collision mesh filename=CAD/electronics.stl scale=0.001 0.001 0.001; visual mesh filename=CAD/electronics.stl scale=0.001 0.001 0.001
- link battery: mass 0.19006392383638834 -> 0.18315250842415606
Joints:
- removed joint base_base_cover
- removed joint base_cover_battery
- removed joint base_mounting_plate
- added joint base_battery_mount: type fixed, parent base, child battery_mount, origin xyz=-1.8325866024682113e-09 0.06599999759782552 -3.6152415994195054e-09 rpy=-3.1415926535897927 1.883898413669496e-21 3.066991105526992e-15
- added joint base_electronics: type fixed, parent base, child electronics, origin xyz=-0.03263500183258655 0.057999997597825405 0.013999996384758396 rpy=3.1415926535897927 -1.883898413669496e-21 -3.14159265358979
- added joint battery_mount_battery: type fixed, parent battery_mount, child battery, origin xyz=0.0 0.06600000000000002 0.0020000000000000018 rpy=1.4836778140138092e-67 -3.76158192263132e-37 3.141592653589793
- added joint camera_mount_camera: type fixed, parent camera_mount, child camera, origin xyz=-0.017824999999999997 0.006999999999999993 0.009474999999999997 rpy=1.5707963267948966 -0.0 -2.574953536144704e-36
- added joint electronics_camera_mount: type fixed, parent electronics, child camera_mount, origin xyz=-0.004340000000000002 0.003940000000000019 -0.012240000000000003 rpy=1.483687499912472e-67 -3.76158192263132e-37 -3.9442911284505303e-31
