Commit message: Split printed parts and hardware into two separate folders

File: hexapod.urdf (robot description, URDF)
Before this commit: robot Hexapod, 72 links, 71 joints
Links:
- link base: geometry collision mesh filename=CAD/printed_parts/base.stl scale=0.001 0.001 0.001; visual mesh filename=CAD/printed_parts/base.stl scale=0.001 0.001 0.001
- link battery: geometry collision mesh filename=CAD/hardware/battery.stl scale=0.001 0.001 0.001; visual mesh filename=CAD/hardware/battery.stl scale=0.001 0.001 0.001
- link battery_mount: geometry collision mesh filename=CAD/printed_parts/battery_mount.stl scale=0.001 0.001 0.001; visual mesh filename=CAD/printed_parts/battery_mount.stl scale=0.001 0.001 0.001
- link camera: geometry collision mesh filename=CAD/hardware/camera.stl scale=0.001 0.001 0.001; visual mesh filename=CAD/hardware/camera.stl scale=0.001 0.001 0.001
- link camera_mount: geometry collision mesh filename=CAD/printed_parts/camera_mount.stl scale=0.001 0.001 0.001; visual mesh filename=CAD/printed_parts/camera_mount.stl scale=0.001 0.001 0.001
- link electronics: geometry collision mesh filename=CAD/hardware/electronics.stl scale=0.001 0.001 0.001; visual mesh filename=CAD/hardware/electronics.stl scale=0.001 0.001 0.001
- link leg_1_coxa_bracket_A: geometry collision mesh filename=CAD/printed_parts/bracket_A.stl scale=0.001 0.001 0.001; visual mesh filename=CAD/printed_parts/bracket_A.stl scale=0.001 0.001 0.001
- link leg_1_coxa_bracket_B: geometry collision mesh filename=CAD/printed_parts/bracket_B.stl scale=0.001 0.001 0.001; visual mesh filename=CAD/printed_parts/bracket_B.stl scale=0.001 0.001 0.001
- link leg_1_coxa_motor: geometry collision mesh filename=CAD/hardware/MG996R.stl scale=0.001 0.001 0.001; visual mesh filename=CAD/hardware/MG996R.stl scale=0.001 0.001 0.001
- link leg_1_femur: geometry collision mesh filename=CAD/printed_parts/femur.stl scale=0.001 0.001 0.001; visual mesh filename=CAD/printed_parts/femur.stl scale=0.001 0.001 0.001
- link leg_1_femur_bracket_A: geometry collision mesh filename=CAD/printed_parts/bracket_A.stl scale=0.001 0.001 0.001; visual mesh filename=CAD/printed_parts/bracket_A.stl scale=0.001 0.001 0.001
- link leg_1_femur_bracket_B: geometry collision mesh filename=CAD/printed_parts/bracket_B.stl scale=0.001 0.001 0.001; visual mesh filename=CAD/printed_parts/bracket_B.stl scale=0.001 0.001 0.001
- link leg_1_femur_motor: geometry collision mesh filename=CAD/hardware/MG996R.stl scale=0.001 0.001 0.001; visual mesh filename=CAD/hardware/MG996R.stl scale=0.001 0.001 0.001
- link leg_1_tibia: geometry collision mesh filename=CAD/printed_parts/tibia.stl scale=0.001 0.001 0.001; visual mesh filename=CAD/printed_parts/tibia.stl scale=0.001 0.001 0.001
- link leg_1_tibia_bracket_A: geometry collision mesh filename=CAD/printed_parts/bracket_A.stl scale=0.001 0.001 0.001; visual mesh filename=CAD/printed_parts/bracket_A.stl scale=0.001 0.001 0.001
- link leg_1_tibia_bracket_B: geometry collision mesh filename=CAD/printed_parts/bracket_B.stl scale=0.001 0.001 0.001; visual mesh filename=CAD/printed_parts/bracket_B.stl scale=0.001 0.001 0.001
- link leg_1_tibia_motor: geometry collision mesh filename=CAD/hardware/MG996R.stl scale=0.001 0.001 0.001; visual mesh filename=CAD/hardware/MG996R.stl scale=0.001 0.001 0.001
- link leg_2_coxa_bracket_A: geometry collision mesh filename=CAD/printed_parts/bracket_A.stl scale=0.001 0.001 0.001; visual mesh filename=CAD/printed_parts/bracket_A.stl scale=0.001 0.001 0.001
- link leg_2_coxa_bracket_B: geometry collision mesh filename=CAD/printed_parts/bracket_B.stl scale=0.001 0.001 0.001; visual mesh filename=CAD/printed_parts/bracket_B.stl scale=0.001 0.001 0.001
- link leg_2_coxa_motor: geometry collision mesh filename=CAD/hardware/MG996R.stl scale=0.001 0.001 0.001; visual mesh filename=CAD/hardware/MG996R.stl scale=0.001 0.001 0.001
- link leg_2_femur: geometry collision mesh filename=CAD/printed_parts/femur.stl scale=0.001 0.001 0.001; visual mesh filename=CAD/printed_parts/femur.stl scale=0.001 0.001 0.001
- link leg_2_femur_bracket_A: geometry collision mesh filename=CAD/printed_parts/bracket_A.stl scale=0.001 0.001 0.001; visual mesh filename=CAD/printed_parts/bracket_A.stl scale=0.001 0.001 0.001
- link leg_2_femur_bracket_B: geometry collision mesh filename=CAD/printed_parts/bracket_B.stl scale=0.001 0.001 0.001; visual mesh filename=CAD/printed_parts/bracket_B.stl scale=0.001 0.001 0.001
- link leg_2_femur_motor: geometry collision mesh filename=CAD/hardware/MG996R.stl scale=0.001 0.001 0.001; visual mesh filename=CAD/hardware/MG996R.stl scale=0.001 0.001 0.001
- link leg_2_tibia: geometry collision mesh filename=CAD/printed_parts/tibia.stl scale=0.001 0.001 0.001; visual mesh filename=CAD/printed_parts/tibia.stl scale=0.001 0.001 0.001
- link leg_2_tibia_bracket_A: geometry collision mesh filename=CAD/printed_parts/bracket_A.stl scale=0.001 0.001 0.001; visual mesh filename=CAD/printed_parts/bracket_A.stl scale=0.001 0.001 0.001
- link leg_2_tibia_bracket_B: geometry collision mesh filename=CAD/printed_parts/bracket_B.stl scale=0.001 0.001 0.001; visual mesh filename=CAD/printed_parts/bracket_B.stl scale=0.001 0.001 0.001
- link leg_2_tibia_motor: geometry collision mesh filename=CAD/hardware/MG996R.stl scale=0.001 0.001 0.001; visual mesh filename=CAD/hardware/MG996R.stl scale=0.001 0.001 0.001
- link leg_3_coxa_bracket_A: geometry collision mesh filename=CAD/printed_parts/bracket_A.stl scale=0.001 0.001 0.001; visual mesh filename=CAD/printed_parts/bracket_A.stl scale=0.001 0.001 0.001
- link leg_3_coxa_bracket_B: geometry collision mesh filename=CAD/printed_parts/bracket_B.stl scale=0.001 0.001 0.001; visual mesh filename=CAD/printed_parts/bracket_B.stl scale=0.001 0.001 0.001
- link leg_3_coxa_motor: geometry collision mesh filename=CAD/hardware/MG996R.stl scale=0.001 0.001 0.001; visual mesh filename=CAD/hardware/MG996R.stl scale=0.001 0.001 0.001
- link leg_3_femur: geometry collision mesh filename=CAD/printed_parts/femur.stl scale=0.001 0.001 0.001; visual mesh filename=CAD/printed_parts/femur.stl scale=0.001 0.001 0.001
- link leg_3_femur_bracket_A: geometry collision mesh filename=CAD/printed_parts/bracket_A.stl scale=0.001 0.001 0.001; visual mesh filename=CAD/printed_parts/bracket_A.stl scale=0.001 0.001 0.001
- link leg_3_femur_bracket_B: geometry collision mesh filename=CAD/printed_parts/bracket_B.stl scale=0.001 0.001 0.001; visual mesh filename=CAD/printed_parts/bracket_B.stl scale=0.001 0.001 0.001
- link leg_3_femur_motor: geometry collision mesh filename=CAD/hardware/MG996R.stl scale=0.001 0.001 0.001; visual mesh filename=CAD/hardware/MG996R.stl scale=0.001 0.001 0.001
- link leg_3_tibia: geometry collision mesh filename=CAD/printed_parts/tibia.stl scale=0.001 0.001 0.001; visual mesh filename=CAD/printed_parts/tibia.stl scale=0.001 0.001 0.001
- link leg_3_tibia_bracket_A: geometry collision mesh filename=CAD/printed_parts/bracket_A.stl scale=0.001 0.001 0.001; visual mesh filename=CAD/printed_parts/bracket_A.stl scale=0.001 0.001 0.001
- link leg_3_tibia_bracket_B: geometry collision mesh filename=CAD/printed_parts/bracket_B.stl scale=0.001 0.001 0.001; visual mesh filename=CAD/printed_parts/bracket_B.stl scale=0.001 0.001 0.001
- link leg_3_tibia_motor: geometry collision mesh filename=CAD/hardware/MG996R.stl scale=0.001 0.001 0.001; visual mesh filename=CAD/hardware/MG996R.stl scale=0.001 0.001 0.001
- link leg_4_coxa_bracket_A: geometry collision mesh filename=CAD/printed_parts/bracket_A.stl scale=0.001 0.001 0.001; visual mesh filename=CAD/printed_parts/bracket_A.stl scale=0.001 0.001 0.001
- link leg_4_coxa_bracket_B: geometry collision mesh filename=CAD/printed_parts/bracket_B.stl scale=0.001 0.001 0.001; visual mesh filename=CAD/printed_parts/bracket_B.stl scale=0.001 0.001 0.001
- link leg_4_coxa_motor: geometry collision mesh filename=CAD/hardware/MG996R.stl scale=0.001 0.001 0.001; visual mesh filename=CAD/hardware/MG996R.stl scale=0.001 0.001 0.001
- link leg_4_femur: geometry collision mesh filename=CAD/printed_parts/femur.stl scale=0.001 0.001 0.001; visual mesh filename=CAD/printed_parts/femur.stl scale=0.001 0.001 0.001
- link leg_4_femur_bracket_A: geometry collision mesh filename=CAD/printed_parts/bracket_A.stl scale=0.001 0.001 0.001; visual mesh filename=CAD/printed_parts/bracket_A.stl scale=0.001 0.001 0.001
- link leg_4_femur_bracket_B: geometry collision mesh filename=CAD/printed_parts/bracket_B.stl scale=0.001 0.001 0.001; visual mesh filename=CAD/printed_parts/bracket_B.stl scale=0.001 0.001 0.001
- link leg_4_femur_motor: geometry collision mesh filename=CAD/hardware/MG996R.stl scale=0.001 0.001 0.001; visual mesh filename=CAD/hardware/MG996R.stl scale=0.001 0.001 0.001
- link leg_4_tibia: geometry collision mesh filename=CAD/printed_parts/tibia.stl scale=0.001 0.001 0.001; visual mesh filename=CAD/printed_parts/tibia.stl scale=0.001 0.001 0.001
- link leg_4_tibia_bracket_A: geometry collision mesh filename=CAD/printed_parts/bracket_A.stl scale=0.001 0.001 0.001; visual mesh filename=CAD/printed_parts/bracket_A.stl scale=0.001 0.001 0.001
- link leg_4_tibia_bracket_B: geometry collision mesh filename=CAD/printed_parts/bracket_B.stl scale=0.001 0.001 0.001; visual mesh filename=CAD/printed_parts/bracket_B.stl scale=0.001 0.001 0.001
- link leg_4_tibia_motor: geometry collision mesh filename=CAD/hardware/MG996R.stl scale=0.001 0.001 0.001; visual mesh filename=CAD/hardware/MG996R.stl scale=0.001 0.001 0.001
- link leg_5_coxa_bracket_A: geometry collision mesh filename=CAD/printed_parts/bracket_A.stl scale=0.001 0.001 0.001; visual mesh filename=CAD/printed_parts/bracket_A.stl scale=0.001 0.001 0.001
- link leg_5_coxa_bracket_B: geometry collision mesh filename=CAD/printed_parts/bracket_B.stl scale=0.001 0.001 0.001; visual mesh filename=CAD/printed_parts/bracket_B.stl scale=0.001 0.001 0.001
- link leg_5_coxa_motor: geometry collision mesh filename=CAD/hardware/MG996R.stl scale=0.001 0.001 0.001; visual mesh filename=CAD/hardware/MG996R.stl scale=0.001 0.001 0.001
- link leg_5_femur: geometry collision mesh filename=CAD/printed_parts/femur.stl scale=0.001 0.001 0.001; visual mesh filename=CAD/printed_parts/femur.stl scale=0.001 0.001 0.001
- link leg_5_femur_bracket_A: geometry collision mesh filename=CAD/printed_parts/bracket_A.stl scale=0.001 0.001 0.001; visual mesh filename=CAD/printed_parts/bracket_A.stl scale=0.001 0.001 0.001
- link leg_5_femur_bracket_B: geometry collision mesh filename=CAD/printed_parts/bracket_B.stl scale=0.001 0.001 0.001; visual mesh filename=CAD/printed_parts/bracket_B.stl scale=0.001 0.001 0.001
- link leg_5_femur_motor: geometry collision mesh filename=CAD/hardware/MG996R.stl scale=0.001 0.001 0.001; visual mesh filename=CAD/hardware/MG996R.stl scale=0.001 0.001 0.001
- link leg_5_tibia: geometry collision mesh filename=CAD/printed_parts/tibia.stl scale=0.001 0.001 0.001; visual mesh filename=CAD/printed_parts/tibia.stl scale=0.001 0.001 0.001
- link leg_5_tibia_bracket_A: geometry collision mesh filename=CAD/printed_parts/bracket_A.stl scale=0.001 0.001 0.001; visual mesh filename=CAD/printed_parts/bracket_A.stl scale=0.001 0.001 0.001
- link leg_5_tibia_bracket_B: geometry collision mesh filename=CAD/printed_parts/bracket_B.stl scale=0.001 0.001 0.001; visual mesh filename=CAD/printed_parts/bracket_B.stl scale=0.001 0.001 0.001
- link leg_5_tibia_motor: geometry collision mesh filename=CAD/hardware/MG996R.stl scale=0.001 0.001 0.001; visual mesh filename=CAD/hardware/MG996R.stl scale=0.001 0.001 0.001
- link leg_6_coxa_bracket_A: geometry collision mesh filename=CAD/printed_parts/bracket_A.stl scale=0.001 0.001 0.001; visual mesh filename=CAD/printed_parts/bracket_A.stl scale=0.001 0.001 0.001
- link leg_6_coxa_bracket_B: geometry collision mesh filename=CAD/printed_parts/bracket_B.stl scale=0.001 0.001 0.001; visual mesh filename=CAD/printed_parts/bracket_B.stl scale=0.001 0.001 0.001
- link leg_6_coxa_motor: geometry collision mesh filename=CAD/hardware/MG996R.stl scale=0.001 0.001 0.001; visual mesh filename=CAD/hardware/MG996R.stl scale=0.001 0.001 0.001
- link leg_6_femur: geometry collision mesh filename=CAD/printed_parts/femur.stl scale=0.001 0.001 0.001; visual mesh filename=CAD/printed_parts/femur.stl scale=0.001 0.001 0.001
- link leg_6_femur_bracket_A: geometry collision mesh filename=CAD/printed_parts/bracket_A.stl scale=0.001 0.001 0.001; visual mesh filename=CAD/printed_parts/bracket_A.stl scale=0.001 0.001 0.001
- link leg_6_femur_bracket_B: geometry collision mesh filename=CAD/printed_parts/bracket_B.stl scale=0.001 0.001 0.001; visual mesh filename=CAD/printed_parts/bracket_B.stl scale=0.001 0.001 0.001
- link leg_6_femur_motor: geometry collision mesh filename=CAD/hardware/MG996R.stl scale=0.001 0.001 0.001; visual mesh filename=CAD/hardware/MG996R.stl scale=0.001 0.001 0.001
- link leg_6_tibia: geometry collision mesh filename=CAD/printed_parts/tibia.stl scale=0.001 0.001 0.001; visual mesh filename=CAD/printed_parts/tibia.stl scale=0.001 0.001 0.001
- link leg_6_tibia_bracket_A: geometry collision mesh filename=CAD/printed_parts/bracket_A.stl scale=0.001 0.001 0.001; visual mesh filename=CAD/printed_parts/bracket_A.stl scale=0.001 0.001 0.001
- link leg_6_tibia_bracket_B: geometry collision mesh filename=CAD/printed_parts/bracket_B.stl scale=0.001 0.001 0.001; visual mesh filename=CAD/printed_parts/bracket_B.stl scale=0.001 0.001 0.001
- link leg_6_tibia_motor: geometry collision mesh filename=CAD/hardware/MG996R.stl scale=0.001 0.001 0.001; visual mesh filename=CAD/hardware/MG996R.stl scale=0.001 0.001 0.001

Commit message: Fixed weird bug with inertia coefficients for leg 2 being off

File: hexapod.urdf (robot description, URDF)
Before this commit: robot Hexapod, 72 links, 71 joints
Links:
- link leg_2_coxa_bracket_A: mass 0.09291760132314016 -> 0.01302030082235085
- link leg_2_coxa_bracket_B: mass 0.029476964029288902 -> 0.004130529991365324
- link leg_2_coxa_motor: mass 0.20795327871559424 -> 0.029139949883713843
- link leg_2_femur: mass 0.155588084324102 -> 0.021802151943504742
- link leg_2_femur_bracket_A: mass 0.09291760132314016 -> 0.01302030082235085
- link leg_2_femur_bracket_B: mass 0.029476964029288902 -> 0.004130529991365324
- link leg_2_femur_motor: mass 0.20795327871559424 -> 0.029139949883713843
- link leg_2_tibia: mass 0.16010206435140967 -> 0.02243468417663065
- link leg_2_tibia_bracket_A: mass 0.09291760132314016 -> 0.01302030082235085
- link leg_2_tibia_bracket_B: mass 0.029476964029288902 -> 0.004130529991365324
- link leg_2_tibia_motor: mass 0.20795327871559424 -> 0.029139949883713843

Commit message: Removed camera -> now optional

File: hexapod.urdf (robot description, URDF)
Before this commit: robot Hexapod, 72 links, 71 joints
Links:
- removed link camera
- removed link camera_mount
Joints:
- removed joint camera_mount_camera
- removed joint electronics_camera_mount

Commit message: Added stiffeners

File: hexapod.urdf (robot description, URDF)
Before this commit: robot Hexapod, 70 links, 69 joints
Links:
- added link bottom_stiffeners, mass 0.04994655381225562; collision mesh filename=CAD/printed_parts/bottom_stiffeners.stl scale=0.001 0.001 0.001; visual mesh filename=CAD/printed_parts/bottom_stiffeners.stl scale=0.001 0.001 0.001
- added link top_stiffeners, mass 0.01808559434559243; collision mesh filename=CAD/printed_parts/top_stiffeners.stl scale=0.001 0.001 0.001; visual mesh filename=CAD/printed_parts/top_stiffeners.stl scale=0.001 0.001 0.001
Joints:
- added joint battery_mount_bottom_stiffeners: type fixed, parent battery_mount, child bottom_stiffeners, origin xyz=-0.030634999999999996 0.013999999999999986 0.0020000000000000018 rpy=1.4836778140138092e-67 -3.76158192263132e-37 3.141592653589793
- added joint electronics_top_stiffeners: type fixed, parent electronics, child top_stiffeners, origin xyz=0.0 0.0 -0.0012000000000000012 rpy=2.7755575615628914e-17 -3.76158192263132e-37 -3.9442911284505303e-31
