Commit message: New version, kind of

File: hexapod.urdf (robot description, URDF)
Before this commit: robot Hexapod, 72 links, 71 joints
Links:
- link base: geometry collision mesh filename=CAD/stl/parts/base.stl scale=0.001 0.001 0.001; visual mesh filename=CAD/stl/parts/base.stl scale=0.001 0.001 0.001
- link battery: geometry collision mesh filename=CAD/stl/hardware/battery.stl scale=0.001 0.001 0.001; visual mesh filename=CAD/stl/hardware/battery.stl scale=0.001 0.001 0.001
- link battery_mount: geometry collision mesh filename=CAD/stl/parts/battery_mount.stl scale=0.001 0.001 0.001; visual mesh filename=CAD/stl/parts/battery_mount.stl scale=0.001 0.001 0.001
- link bottom_stiffeners: geometry collision mesh filename=CAD/stl/parts/bottom_stiffeners.stl scale=0.001 0.001 0.001; visual mesh filename=CAD/stl/parts/bottom_stiffeners.stl scale=0.001 0.001 0.001
- link electronics: geometry collision mesh filename=CAD/stl/hardware/electronics.stl scale=0.001 0.001 0.001; visual mesh filename=CAD/stl/hardware/electronics.stl scale=0.001 0.001 0.001
- link leg_1_coxa_bracket_A: geometry collision mesh filename=CAD/stl/parts/bracket_A.stl scale=0.001 0.001 0.001; visual mesh filename=CAD/stl/parts/bracket_A.stl scale=0.001 0.001 0.001
- link leg_1_coxa_bracket_B: geometry collision mesh filename=CAD/stl/parts/bracket_B.stl scale=0.001 0.001 0.001; visual mesh filename=CAD/stl/parts/bracket_B.stl scale=0.001 0.001 0.001
- link leg_1_coxa_motor: geometry collision mesh filename=CAD/stl/hardware/MG996R.stl scale=0.001 0.001 0.001; visual mesh filename=CAD/stl/hardware/MG996R.stl scale=0.001 0.001 0.001
- link leg_1_femur: geometry collision mesh filename=CAD/stl/parts/femur.stl scale=0.001 0.001 0.001; visual mesh filename=CAD/stl/parts/femur.stl scale=0.001 0.001 0.001
- link leg_1_femur_bracket_A: geometry collision mesh filename=CAD/stl/parts/bracket_A.stl scale=0.001 0.001 0.001; visual mesh filename=CAD/stl/parts/bracket_A.stl scale=0.001 0.001 0.001
- link leg_1_femur_bracket_B: geometry collision mesh filename=CAD/stl/parts/bracket_B.stl scale=0.001 0.001 0.001; visual mesh filename=CAD/stl/parts/bracket_B.stl scale=0.001 0.001 0.001
- link leg_1_femur_motor: geometry collision mesh filename=CAD/stl/hardware/MG996R.stl scale=0.001 0.001 0.001; visual mesh filename=CAD/stl/hardware/MG996R.stl scale=0.001 0.001 0.001
- link leg_1_tibia: geometry collision mesh filename=CAD/stl/parts/tibia.stl scale=0.001 0.001 0.001; visual mesh filename=CAD/stl/parts/tibia.stl scale=0.001 0.001 0.001
- link leg_1_tibia_bracket_A: geometry collision mesh filename=CAD/stl/parts/bracket_A.stl scale=0.001 0.001 0.001; visual mesh filename=CAD/stl/parts/bracket_A.stl scale=0.001 0.001 0.001
- link leg_1_tibia_bracket_B: geometry collision mesh filename=CAD/stl/parts/bracket_B.stl scale=0.001 0.001 0.001; visual mesh filename=CAD/stl/parts/bracket_B.stl scale=0.001 0.001 0.001
- link leg_1_tibia_motor: geometry collision mesh filename=CAD/stl/hardware/MG996R.stl scale=0.001 0.001 0.001; visual mesh filename=CAD/stl/hardware/MG996R.stl scale=0.001 0.001 0.001
- link leg_2_coxa_bracket_A: geometry collision mesh filename=CAD/stl/parts/bracket_A.stl scale=0.001 0.001 0.001; visual mesh filename=CAD/stl/parts/bracket_A.stl scale=0.001 0.001 0.001
- link leg_2_coxa_bracket_B: geometry collision mesh filename=CAD/stl/parts/bracket_B.stl scale=0.001 0.001 0.001; visual mesh filename=CAD/stl/parts/bracket_B.stl scale=0.001 0.001 0.001
- link leg_2_coxa_motor: geometry collision mesh filename=CAD/stl/hardware/MG996R.stl scale=0.001 0.001 0.001; visual mesh filename=CAD/stl/hardware/MG996R.stl scale=0.001 0.001 0.001
- link leg_2_femur: geometry collision mesh filename=CAD/stl/parts/femur.stl scale=0.001 0.001 0.001; visual mesh filename=CAD/stl/parts/femur.stl scale=0.001 0.001 0.001
- link leg_2_femur_bracket_A: geometry collision mesh filename=CAD/stl/parts/bracket_A.stl scale=0.001 0.001 0.001; visual mesh filename=CAD/stl/parts/bracket_A.stl scale=0.001 0.001 0.001
- link leg_2_femur_bracket_B: geometry collision mesh filename=CAD/stl/parts/bracket_B.stl scale=0.001 0.001 0.001; visual mesh filename=CAD/stl/parts/bracket_B.stl scale=0.001 0.001 0.001
- link leg_2_femur_motor: geometry collision mesh filename=CAD/stl/hardware/MG996R.stl scale=0.001 0.001 0.001; visual mesh filename=CAD/stl/hardware/MG996R.stl scale=0.001 0.001 0.001
- link leg_2_tibia: geometry collision mesh filename=CAD/stl/parts/tibia.stl scale=0.001 0.001 0.001; visual mesh filename=CAD/stl/parts/tibia.stl scale=0.001 0.001 0.001
- link leg_2_tibia_bracket_A: geometry collision mesh filename=CAD/stl/parts/bracket_A.stl scale=0.001 0.001 0.001; visual mesh filename=CAD/stl/parts/bracket_A.stl scale=0.001 0.001 0.001
- link leg_2_tibia_bracket_B: geometry collision mesh filename=CAD/stl/parts/bracket_B.stl scale=0.001 0.001 0.001; visual mesh filename=CAD/stl/parts/bracket_B.stl scale=0.001 0.001 0.001
- link leg_2_tibia_motor: geometry collision mesh filename=CAD/stl/hardware/MG996R.stl scale=0.001 0.001 0.001; visual mesh filename=CAD/stl/hardware/MG996R.stl scale=0.001 0.001 0.001
- link leg_3_coxa_bracket_A: geometry collision mesh filename=CAD/stl/parts/bracket_A.stl scale=0.001 0.001 0.001; visual mesh filename=CAD/stl/parts/bracket_A.stl scale=0.001 0.001 0.001
- link leg_3_coxa_bracket_B: geometry collision mesh filename=CAD/stl/parts/bracket_B.stl scale=0.001 0.001 0.001; visual mesh filename=CAD/stl/parts/bracket_B.stl scale=0.001 0.001 0.001
- link leg_3_coxa_motor: geometry collision mesh filename=CAD/stl/hardware/MG996R.stl scale=0.001 0.001 0.001; visual mesh filename=CAD/stl/hardware/MG996R.stl scale=0.001 0.001 0.001
- link leg_3_femur: geometry collision mesh filename=CAD/stl/parts/femur.stl scale=0.001 0.001 0.001; visual mesh filename=CAD/stl/parts/femur.stl scale=0.001 0.001 0.001
- link leg_3_femur_bracket_A: geometry collision mesh filename=CAD/stl/parts/bracket_A.stl scale=0.001 0.001 0.001; visual mesh filename=CAD/stl/parts/bracket_A.stl scale=0.001 0.001 0.001
- link leg_3_femur_bracket_B: geometry collision mesh filename=CAD/stl/parts/bracket_B.stl scale=0.001 0.001 0.001; visual mesh filename=CAD/stl/parts/bracket_B.stl scale=0.001 0.001 0.001
- link leg_3_femur_motor: geometry collision mesh filename=CAD/stl/hardware/MG996R.stl scale=0.001 0.001 0.001; visual mesh filename=CAD/stl/hardware/MG996R.stl scale=0.001 0.001 0.001
- link leg_3_tibia: geometry collision mesh filename=CAD/stl/parts/tibia.stl scale=0.001 0.001 0.001; visual mesh filename=CAD/stl/parts/tibia.stl scale=0.001 0.001 0.001
- link leg_3_tibia_bracket_A: geometry collision mesh filename=CAD/stl/parts/bracket_A.stl scale=0.001 0.001 0.001; visual mesh filename=CAD/stl/parts/bracket_A.stl scale=0.001 0.001 0.001
- link leg_3_tibia_bracket_B: geometry collision mesh filename=CAD/stl/parts/bracket_B.stl scale=0.001 0.001 0.001; visual mesh filename=CAD/stl/parts/bracket_B.stl scale=0.001 0.001 0.001
- link leg_3_tibia_motor: geometry collision mesh filename=CAD/stl/hardware/MG996R.stl scale=0.001 0.001 0.001; visual mesh filename=CAD/stl/hardware/MG996R.stl scale=0.001 0.001 0.001
- link leg_4_coxa_bracket_A: geometry collision mesh filename=CAD/stl/parts/bracket_A.stl scale=0.001 0.001 0.001; visual mesh filename=CAD/stl/parts/bracket_A.stl scale=0.001 0.001 0.001
- link leg_4_coxa_bracket_B: geometry collision mesh filename=CAD/stl/parts/bracket_B.stl scale=0.001 0.001 0.001; visual mesh filename=CAD/stl/parts/bracket_B.stl scale=0.001 0.001 0.001
- link leg_4_coxa_motor: geometry collision mesh filename=CAD/stl/hardware/MG996R.stl scale=0.001 0.001 0.001; visual mesh filename=CAD/stl/hardware/MG996R.stl scale=0.001 0.001 0.001
- link leg_4_femur: geometry collision mesh filename=CAD/stl/parts/femur.stl scale=0.001 0.001 0.001; visual mesh filename=CAD/stl/parts/femur.stl scale=0.001 0.001 0.001
- link leg_4_femur_bracket_A: geometry collision mesh filename=CAD/stl/parts/bracket_A.stl scale=0.001 0.001 0.001; visual mesh filename=CAD/stl/parts/bracket_A.stl scale=0.001 0.001 0.001
- link leg_4_femur_bracket_B: geometry collision mesh filename=CAD/stl/parts/bracket_B.stl scale=0.001 0.001 0.001; visual mesh filename=CAD/stl/parts/bracket_B.stl scale=0.001 0.001 0.001
- link leg_4_femur_motor: geometry collision mesh filename=CAD/stl/hardware/MG996R.stl scale=0.001 0.001 0.001; visual mesh filename=CAD/stl/hardware/MG996R.stl scale=0.001 0.001 0.001
- link leg_4_tibia: geometry collision mesh filename=CAD/stl/parts/tibia.stl scale=0.001 0.001 0.001; visual mesh filename=CAD/stl/parts/tibia.stl scale=0.001 0.001 0.001
- link leg_4_tibia_bracket_A: geometry collision mesh filename=CAD/stl/parts/bracket_A.stl scale=0.001 0.001 0.001; visual mesh filename=CAD/stl/parts/bracket_A.stl scale=0.001 0.001 0.001
- link leg_4_tibia_bracket_B: geometry collision mesh filename=CAD/stl/parts/bracket_B.stl scale=0.001 0.001 0.001; visual mesh filename=CAD/stl/parts/bracket_B.stl scale=0.001 0.001 0.001
- link leg_4_tibia_motor: geometry collision mesh filename=CAD/stl/hardware/MG996R.stl scale=0.001 0.001 0.001; visual mesh filename=CAD/stl/hardware/MG996R.stl scale=0.001 0.001 0.001
- link leg_5_coxa_bracket_A: geometry collision mesh filename=CAD/stl/parts/bracket_A.stl scale=0.001 0.001 0.001; visual mesh filename=CAD/stl/parts/bracket_A.stl scale=0.001 0.001 0.001
- link leg_5_coxa_bracket_B: geometry collision mesh filename=CAD/stl/parts/bracket_B.stl scale=0.001 0.001 0.001; visual mesh filename=CAD/stl/parts/bracket_B.stl scale=0.001 0.001 0.001
- link leg_5_coxa_motor: geometry collision mesh filename=CAD/stl/hardware/MG996R.stl scale=0.001 0.001 0.001; visual mesh filename=CAD/stl/hardware/MG996R.stl scale=0.001 0.001 0.001
- link leg_5_femur: geometry collision mesh filename=CAD/stl/parts/femur.stl scale=0.001 0.001 0.001; visual mesh filename=CAD/stl/parts/femur.stl scale=0.001 0.001 0.001
- link leg_5_femur_bracket_A: geometry collision mesh filename=CAD/stl/parts/bracket_A.stl scale=0.001 0.001 0.001; visual mesh filename=CAD/stl/parts/bracket_A.stl scale=0.001 0.001 0.001
- link leg_5_femur_bracket_B: geometry collision mesh filename=CAD/stl/parts/bracket_B.stl scale=0.001 0.001 0.001; visual mesh filename=CAD/stl/parts/bracket_B.stl scale=0.001 0.001 0.001
- link leg_5_femur_motor: geometry collision mesh filename=CAD/stl/hardware/MG996R.stl scale=0.001 0.001 0.001; visual mesh filename=CAD/stl/hardware/MG996R.stl scale=0.001 0.001 0.001
- link leg_5_tibia: geometry collision mesh filename=CAD/stl/parts/tibia.stl scale=0.001 0.001 0.001; visual mesh filename=CAD/stl/parts/tibia.stl scale=0.001 0.001 0.001
- link leg_5_tibia_bracket_A: geometry collision mesh filename=CAD/stl/parts/bracket_A.stl scale=0.001 0.001 0.001; visual mesh filename=CAD/stl/parts/bracket_A.stl scale=0.001 0.001 0.001
- link leg_5_tibia_bracket_B: geometry collision mesh filename=CAD/stl/parts/bracket_B.stl scale=0.001 0.001 0.001; visual mesh filename=CAD/stl/parts/bracket_B.stl scale=0.001 0.001 0.001
- link leg_5_tibia_motor: geometry collision mesh filename=CAD/stl/hardware/MG996R.stl scale=0.001 0.001 0.001; visual mesh filename=CAD/stl/hardware/MG996R.stl scale=0.001 0.001 0.001
- link leg_6_coxa_bracket_A: geometry collision mesh filename=CAD/stl/parts/bracket_A.stl scale=0.001 0.001 0.001; visual mesh filename=CAD/stl/parts/bracket_A.stl scale=0.001 0.001 0.001
- link leg_6_coxa_bracket_B: geometry collision mesh filename=CAD/stl/parts/bracket_B.stl scale=0.001 0.001 0.001; visual mesh filename=CAD/stl/parts/bracket_B.stl scale=0.001 0.001 0.001
- link leg_6_coxa_motor: geometry collision mesh filename=CAD/stl/hardware/MG996R.stl scale=0.001 0.001 0.001; visual mesh filename=CAD/stl/hardware/MG996R.stl scale=0.001 0.001 0.001
- link leg_6_femur: geometry collision mesh filename=CAD/stl/parts/femur.stl scale=0.001 0.001 0.001; visual mesh filename=CAD/stl/parts/femur.stl scale=0.001 0.001 0.001
- link leg_6_femur_bracket_A: geometry collision mesh filename=CAD/stl/parts/bracket_A.stl scale=0.001 0.001 0.001; visual mesh filename=CAD/stl/parts/bracket_A.stl scale=0.001 0.001 0.001
- link leg_6_femur_bracket_B: geometry collision mesh filename=CAD/stl/parts/bracket_B.stl scale=0.001 0.001 0.001; visual mesh filename=CAD/stl/parts/bracket_B.stl scale=0.001 0.001 0.001
- link leg_6_femur_motor: geometry collision mesh filename=CAD/stl/hardware/MG996R.stl scale=0.001 0.001 0.001; visual mesh filename=CAD/stl/hardware/MG996R.stl scale=0.001 0.001 0.001
- link leg_6_tibia: geometry collision mesh filename=CAD/stl/parts/tibia.stl scale=0.001 0.001 0.001; visual mesh filename=CAD/stl/parts/tibia.stl scale=0.001 0.001 0.001
- link leg_6_tibia_bracket_A: geometry collision mesh filename=CAD/stl/parts/bracket_A.stl scale=0.001 0.001 0.001; visual mesh filename=CAD/stl/parts/bracket_A.stl scale=0.001 0.001 0.001
- link leg_6_tibia_bracket_B: geometry collision mesh filename=CAD/stl/parts/bracket_B.stl scale=0.001 0.001 0.001; visual mesh filename=CAD/stl/parts/bracket_B.stl scale=0.001 0.001 0.001
- link leg_6_tibia_motor: geometry collision mesh filename=CAD/stl/hardware/MG996R.stl scale=0.001 0.001 0.001; visual mesh filename=CAD/stl/hardware/MG996R.stl scale=0.001 0.001 0.001
- link top_stiffeners: geometry collision mesh filename=CAD/stl/parts/top_stiffeners.stl scale=0.001 0.001 0.001; visual mesh filename=CAD/stl/parts/top_stiffeners.stl scale=0.001 0.001 0.001
